File: Vanguard 2.3 production files + duplicates/Vanguard_new.kicad_sch (KiCad schematic)
At the start: 91 parts, among them J1 USB_C_Receptacle_USB2.0_16P, J2 Conn_02x03_Pin, J3 Micro_SD_Card_Det1, J4 STARBOARD_SERVO, J5 PORTSIDE_SERVO, J6 Battery In, J7 EJECTION_SERVO, Q1 BSS138, Q2 BSS138, Q3 BSS138, Q4 BSS138, U1 ATSAMD11D14A-M, U10 BMP390L, U2 ATmega4809-A, U3 AT25DF641A-SH-T, U4 AP2112K-3.3, U5 BD1020HFV, U6 BNO086, U7 TXB0104D, U8 TPS61092, U9 MPM3610AGQV-P, Y1 32.768kHz

Commit message: production folder
Parts:
- J1: footprint Connector_USB:USB_C_Receptacle_Amphenol_12401548E4-2A -> Connector_USB:USB_C_Receptacle_GCT_USB4085
- J6: footprint Connector_PinHeader_2.54mm:PinHeader_1x02_P2.54mm_Vertical -> Connector_JST:JST_PH_B2B-PH-K_1x02_P2.00mm_Vertical
Changed lines of the file:
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@@
 	(label "RX_UPDI"
 		(at 153.67 50.8 0)
+		(fields_autoplaced yes)
 		(effects
 			(font
@@
 	(label "TX_UPDI"
 		(at 153.67 48.26 0)
+		(fields_autoplaced yes)
 		(effects
 			(font
@@
 			)
 		)
-		(property "Footprint" "Connector_PinHeader_2.54mm:PinHeader_1x02_P2.54mm_Vertical"
+		(property "Footprint" "Connector_JST:JST_PH_B2B-PH-K_1x02_P2.00mm_Vertical"
 			(at 334.01 163.83 0)
 			(effects
@@
 			)
 		)
-		(property "Footprint" "Connector_USB:USB_C_Receptacle_Amphenol_12401548E4-2A"
+		(property "Footprint" "Connector_USB:USB_C_Receptacle_GCT_USB4085"
 			(at 31.75 39.37 0)
 			(effects
