File: vanguard/2.3.2/Vanguard_new.kicad_sch (KiCad schematic)
At the start: 91 parts, among them J1 USB_C_Receptacle_USB2.0_16P, J2 Conn_02x03_Pin, J3 Micro_SD_Card_Det1, J4 STARBOARD_SERVO, J5 PORTSIDE_SERVO, J6 Battery In, J7 EJECTION_SERVO, Q1 BSS138, Q2 BSS138, Q3 BSS138, Q4 BSS138, U1 ATSAMD11D14A-M, U10 BMP390L, U2 ATmega4809-A, U3 AT25DF641A-SH-T, U4 AP2112K-3.3, U5 BD1020HFV, U6 BNO086, U7 TXB0104D, U8 TPS61092, U9 MPM3610AGQV-P, Y1 32.768kHz

Commit message: 2.3.2 created, 2.4.1 removed
Parts:
- J3: footprint Connector_Card:microSD_HC_Hirose_DM3D-SF -> Connector_Card:microSD_HC_Molex_104031-0811
Changed lines of the file:
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@@
 (kicad_sch
-	(version 20250114)
+	(version 20231120)
 	(generator "eeschema")
-	(generator_version "9.0")
+	(generator_version "8.0")
 	(paper "USLedger")
-	(rectangle
-		(start 12.065 13.335)
-		(end 269.24 100.33)
-		(stroke
-			(width 0)
-			(type default)
-		)
-		(fill
-			(type none)
-		)
-	)
-	(rectangle
-		(start 12.7 100.33)
-		(end 189.23 193.04)
-		(stroke
-			(width 0)
-			(type default)
-		)
-		(fill
-			(type none)
-		)
-	)
-	(rectangle
-		(start 138.43 193.04)
-		(end 228.6 266.7)
-		(stroke
-			(width 0)
-			(type default)
-		)
-		(fill
-			(type none)
-		)
-	)
-	(rectangle
-		(start 12.7 193.04)
-		(end 138.43 267.335)
-		(stroke
-			(width 0)
-			(type default)
-		)
-		(fill
-			(type none)
-		)
-	)
-	(rectangle
-		(start 269.24 13.97)
-		(end 418.465 77.47)
-		(stroke
-			(width 0)
-			(type default)
-		)
-		(fill
-			(type none)
-		)
-	)
-	(rectangle
-		(start 269.24 77.47)
-		(end 360.68 139.7)
-		(stroke
-			(width 0)
-			(type default)
-		)
-		(fill
-			(type none)
-		)
-	)
-	(text "SD CARD\n"
-		(exclude_from_sim no)
-		(at 108.966 205.994 0)
-		(effects
-			(font
-				(size 2.54 2.54)
-			)
-		)
-	)
-	(text "INPUT USB"
-		(exclude_from_sim no)
-		(at 244.094 22.352 0)
-		(effects
-			(font
-				(size 2.54 2.54)
-			)
-		)
-	)
-	(text "BUZZER\n"
-		(exclude_from_sim no)
-		(at 371.348 88.392 0)
-		(effects
-			(font
-				(size 2.54 2.54)
-			)
-		)
-	)
-	(text "POWER STABILIZATION"
-		(exclude_from_sim no)
-		(at 301.244 22.352 0)
-		(effects
-			(font
-				(size 2.54 2.54)
-			)
-		)
-	)
-	(text "FLASH CHIP\n"
-		(exclude_from_sim no)
-		(at 212.2747 205.1733 0)
-		(effects
-			(font
-				(size 2.54 2.54)
-			)
-		)
-	)
-	(text "SENSORS "
-		(exclude_from_sim no)
-		(at 155.956 109.982 0)
-		(effects
-			(font
-				(size 2.54 2.54)
-			)
-		)
-	)
-	(text "SERVOS\n"
-		(exclude_from_sim no)
-		(at 280.924 146.304 0)
-		(effects
-			(font
-				(size 2.54 2.54)
-			)
-		)
-	)
-	(text "LEDS\n"
-		(exclude_from_sim no)
-		(at 278.892 87.63 0)
-		(effects
-			(font
-				(size 2.54 2.54)
-			)
-		)
-	)
-	(text "SERVO POWER\n\n"
-		(exclude_from_sim no)
-		(at 339.852 147.066 0)
-		(effects
-			(font
-				(size 2.54 2.54)
-			)
-		)
-	)
 	(junction
 		(at 162.56 48.26)
@@
 		)
 	)
+	(rectangle
+		(start 12.065 13.335)
+		(end 269.24 100.33)
+		(stroke
+			(width 0)
+			(type default)
+		)
+		(fill
+			(type none)
+		)
+	)
+	(rectangle
+		(start 12.7 100.33)
+		(end 189.23 193.04)
+		(stroke
+			(width 0)
+			(type default)
+		)
+		(fill
+			(type none)
+		)
+	)
+	(rectangle
+		(start 138.43 193.04)
+		(end 228.6 266.7)
+		(stroke
+			(width 0)
+			(type default)
+		)
+		(fill
+			(type none)
+		)
+	)
+	(rectangle
+		(start 12.7 193.04)
+		(end 138.43 267.335)
+		(stroke
+			(width 0)
+			(type default)
+		)
+		(fill
+			(type none)
+		)
+	)
+	(rectangle
+		(start 269.24 13.97)
+		(end 418.465 77.47)
+		(stroke
+			(width 0)
+			(type default)
+		)
+		(fill
+			(type none)
+		)
+	)
+	(rectangle
+		(start 269.24 77.47)
+		(end 360.68 139.7)
+		(stroke
+			(width 0)
+			(type default)
+		)
+		(fill
+			(type none)
+		)
+	)
+	(text "SD CARD\n"
+		(exclude_from_sim no)
+		(at 108.966 205.994 0)
+		(effects
+			(font
+				(size 2.54 2.54)
+			)
+		)
+	)
+	(text "INPUT USB"
+		(exclude_from_sim no)
+		(at 244.094 22.352 0)
+		(effects
+			(font
+				(size 2.54 2.54)
+			)
+		)
+	)
+	(text "BUZZER\n"
+		(exclude_from_sim no)
+		(at 371.348 88.392 0)
+		(effects
+			(font
+				(size 2.54 2.54)
+			)
+		)
+	)
+	(text "POWER STABILIZATION"
+		(exclude_from_sim no)
+		(at 301.244 22.352 0)
+		(effects
+			(font
+				(size 2.54 2.54)
+			)
+		)
+	)
+	(text "FLASH CHIP\n"
+		(exclude_from_sim no)
+		(at 212.2747 205.1733 0)
+		(effects
+			(font
+				(size 2.54 2.54)
+			)
+		)
+	)
+	(text "SENSORS "
+		(exclude_from_sim no)
+		(at 155.956 109.982 0)
+		(effects
+			(font
+				(size 2.54 2.54)
+			)
+		)
+	)
+	(text "SERVOS\n"
+		(exclude_from_sim no)
+		(at 280.924 146.304 0)
+		(effects
+			(font
+				(size 2.54 2.54)
+			)
+		)
+	)
+	(text "LEDS\n"
+		(exclude_from_sim no)
+		(at 278.892 87.63 0)
+		(effects
+			(font
+				(size 2.54 2.54)
+			)
+		)
+	)
+	(text "SERVO POWER\n\n"
+		(exclude_from_sim no)
+		(at 339.852 147.066 0)
+		(effects
+			(font
+				(size 2.54 2.54)
+			)
+		)
+	)
 	(label "RX_UPDI"
 		(at 153.67 50.8 0)
@@
 			)
 		)
-		(property "Footprint" "Connector_Card:microSD_HC_Hirose_DM3D-SF"
+		(property "Footprint" "Connector_Card:microSD_HC_Molex_104031-0811"
 			(at 147.32 252.73 0)
 			(effects
@@
 		)
 	)
-	(embedded_fonts no)
 )
