File: vanguard/meddy goof/tardon/tardon/tardon.kicad_sch (KiCad schematic)
At the start: 21 parts, among them Q1 BC817W, U1 STM32F405RGTx, U2 NCP1117-3.3_SOT223, U4 MPU-6000

Commit message: schematic changes
Parts:
- added C11, C12: 100nF, symbol Device:C
- added P1: USB_C_Plug_USB2.0, symbol Connector:USB_C_Plug_USB2.0
- added R10: R, symbol Device:R
- added R11, R8, R9: 10K, symbol Device:R
- added R12, R5: 10k, symbol Device:R
- added R6, R7: 22, symbol Device:R
- added S1: DHT-4235A, DHT-4235A:SW_DHT-4235A, symbol DHT-4235A:DHT-4235A
- added Y1: Crystal_GND2, symbol Device:Crystal_GND2
Connections:
- net +5V is gone; now on net 5V: R2.1
- net 5V USB: now also P1.A4 (VBUS), P1.A9 (VBUS), P1.B4 (VBUS), P1.B9 (VBUS), R8.1
- net GND: now also C11.1, C12.1, P1.A1 (GND), P1.A12 (GND), P1.B1 (GND), P1.B12 (GND), P1.S1 (SHIELD), R10.1, R9.2
- net GYRO_CS: now also U1.20 (PA4), R5.2
- net GYRO_INT: now also U1.24 (PC4)
- net GYRO_SCL: now also U1.21 (PA5)
- net GYRO_SDA: now also U1.23 (PA7)
- net LED1: now also U1.55 (PB3)
- net LED2: now also U1.56 (PB4)
- net UART1_RX: now also U1.42 (PA9)
- net VDD: now also R5.1, S1.3, S1.4
- net RSSI_PAD: now reaches U1.10 (PC2)
- net Current_PAD: now reaches U1.11 (PC3)
- net LED: now reaches U1.14 (PA0)
- net GYRO_SD0: now reaches U1.22 (PA6)
- net GYRO_SD0: now also U4.9 (AD0/SDO)
- net at U1.25 (PC5): now also R8.2, R9.1
- net at U1.31 (VCAP_1): now also C11.2
- net UART6_TX: now reaches U1.37 (PC6)
- net UART6_RX: now reaches U1.38 (PC7)
- net PPM_IN: now reaches U1.40 (PC9)
- net BUZZER: now reaches U1.41 (PA8)
- net UART1_TX: now reaches U1.43 (PA10)
- net at U1.44 (PA11): now also R7.1
- net at U1.45 (PA12): now also R6.1
- net at U1.47 (VCAP_2): now also C12.2
- net at U1.5 (PH0): now also Y1.1
- net at U1.57 (PB5): now also R11.1
- net at U1.58 (PB6): now also R12.1
- net at U1.6 (PH1): now also Y1.3
- net at U1.60 (BOOT0): now also R10.2, S1.1, S1.2
- net VBAT_PAD: now reaches U1.9 (PC1)
- new net: P1.A7 (D-), R7.2
- new net: P1.A6 (D+), R6.2
- new net SCL_PAD: R11.2
- new net SDA_PAD: R12.2
