File: vanguard/board versions/Vang_V2.3.3/_autosave-Vanguard_new.kicad_sch (KiCad schematic)
At the start: 94 parts, among them J1 USB_C_Receptacle_USB2.0_16P, J2 Micro_SD_Card_Det1, J3 Conn_02x03_Odd_Even, J4 Conn_01x03, J5 Conn_01x03, J6 Conn_01x03, J7 Conn_01x02_Pin, Q4 BSS138, U1 TPS82130, U10 ATmega4809-A, U12 AP2112K-3.3, U3 ATSAMD11D14A-M, U4 BMP390L, U5 BD1020HFV-TR, U6 AT25DF641A-SH-T, U8 BNO055, U9 TPS61092, Y1 Crystal

Commit message: dont touch yet
Changed lines of the file:
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@@
+	)
+	(junction
+		(at 180.34 182.88)
+		(diameter 0)
+		(color 0 0 0 0)
 	)
 	(junction
@@
 	)
 	(junction
+		(at 242.57 128.27)
+		(diameter 0)
+		(color 0 0 0 0)
+	)
+	(junction
 		(at 167.64 231.14)
 		(diameter 0)
@@
 	(wire
 		(pts
+			(xy 191.77 190.5) (xy 191.77 179.07)
+		)
+		(stroke
+			(width 0)
+			(type default)
+		)
+	)
+	(wire
+		(pts
 			(xy 168.91 52.07) (xy 171.45 52.07)
 		)
@@
 	(wire
 		(pts
+			(xy 149.86 198.12) (xy 152.4 198.12)
+		)
+		(stroke
+			(width 0)
+			(type default)
+		)
+	)
+	(wire
+		(pts
 			(xy 356.87 167.64) (xy 344.17 167.64)
 		)
@@
 	(wire
 		(pts
+			(xy 152.4 198.12) (xy 219.71 265.43)
+		)
+		(stroke
+			(width 0)
+			(type default)
+		)
+	)
+	(wire
+		(pts
 			(xy 339.09 162.56) (xy 349.25 162.56)
 		)
@@
 	(wire
 		(pts
+			(xy 12.7 190.5) (xy 101.6 101.6)
+		)
+		(stroke
+			(width 0)
+			(type default)
+		)
+	)
+	(wire
+		(pts
 			(xy 205.74 222.25) (xy 205.74 226.06)
 		)
@@
 	(wire
 		(pts
+			(xy 12.7 191.77) (xy 12.7 190.5)
+		)
+		(stroke
+			(width 0)
+			(type default)
+		)
+	)
+	(wire
+		(pts
 			(xy 63.5 147.32) (xy 63.5 149.86)
 		)
@@
 	(wire
 		(pts
+			(xy 242.57 128.27) (xy 266.7 104.14)
+		)
+		(stroke
+			(width 0)
+			(type default)
+		)
+	)
+	(wire
+		(pts
 			(xy 218.44 226.06) (xy 213.36 226.06)
 		)
@@
 	(wire
 		(pts
+			(xy 152.4 264.16) (xy 223.52 193.04)
+		)
+		(stroke
+			(width 0)
+			(type default)
+		)
+	)
+	(wire
+		(pts
 			(xy 171.45 46.99) (xy 170.18 46.99)
 		)
@@
 	(wire
 		(pts
+			(xy 191.77 179.07) (xy 242.57 128.27)
+		)
+		(stroke
+			(width 0)
+			(type default)
+		)
+	)
+	(wire
+		(pts
 			(xy 111.76 38.1) (xy 121.92 38.1)
 		)
@@
 	(wire
 		(pts
+			(xy 15.24 264.16) (xy 83.82 195.58)
+		)
+		(stroke
+			(width 0)
+			(type default)
+		)
+	)
+	(wire
+		(pts
 			(xy 146.05 40.64) (xy 166.37 40.64)
 		)
@@
 	(wire
 		(pts
+			(xy 83.82 195.58) (xy 152.4 264.16)
+		)
+		(stroke
+			(width 0)
+			(type default)
+		)
+	)
+	(wire
+		(pts
 			(xy 172.72 133.35) (xy 175.26 133.35)
 		)
@@
 	(wire
 		(pts
+			(xy 105.41 193.04) (xy 105.41 184.15)
+		)
+		(stroke
+			(width 0)
+			(type default)
+		)
+	)
+	(wire
+		(pts
 			(xy 335.28 40.64) (xy 342.9 40.64)
 		)
@@
 	(wire
 		(pts
+			(xy 189.23 100.33) (xy 189.23 109.22)
+		)
+		(stroke
+			(width 0)
+			(type default)
+		)
+	)
+	(wire
+		(pts
 			(xy 389.89 154.94) (xy 381 154.94)
 		)
@@
 	(wire
 		(pts
+			(xy 54.61 234.95) (xy 83.82 264.16)
+		)
+		(stroke
+			(width 0)
+			(type default)
+		)
+	)
+	(wire
+		(pts
 			(xy 212.09 62.23) (xy 215.9 62.23)
 		)
@@
 	(wire
 		(pts
+			(xy 101.6 104.14) (xy 180.34 182.88)
+		)
+		(stroke
+			(width 0)
+			(type default)
+		)
+	)
+	(wire
+		(pts
 			(xy 92.71 129.54) (xy 92.71 124.46)
 		)
@@
 	(wire
 		(pts
+			(xy 180.34 182.88) (xy 190.5 193.04)
+		)
+		(stroke
+			(width 0)
+			(type default)
+		)
+	)
+	(wire
+		(pts
 			(xy 381 154.94) (xy 377.19 154.94)
 		)
@@
 	(wire
 		(pts
+			(xy 83.82 264.16) (xy 149.86 198.12)
+		)
+		(stroke
+			(width 0)
+			(type default)
+		)
+	)
+	(wire
+		(pts
 			(xy 167.64 72.39) (xy 167.64 54.61)
 		)
@@
 	(wire
 		(pts
+			(xy 12.7 193.04) (xy 54.61 234.95)
+		)
+		(stroke
+			(width 0)
+			(type default)
+		)
+	)
+	(wire
+		(pts
 			(xy 92.71 52.07) (xy 116.84 52.07)
 		)
@@
 	(wire
 		(pts
+			(xy 12.7 100.33) (xy 105.41 193.04)
+		)
+		(stroke
+			(width 0)
+			(type default)
+		)
+	)
+	(wire
+		(pts
 			(xy 349.25 165.1) (xy 356.87 165.1)
 		)
@@
 	(wire
 		(pts
+			(xy 189.23 109.22) (xy 269.24 189.23)
+		)
+		(stroke
+			(width 0)
+			(type default)
+		)
+	)
+	(wire
+		(pts
 			(xy 382.27 102.87) (xy 382.27 105.41)
 		)
@@
 	(wire
 		(pts
+			(xy 101.6 101.6) (xy 101.6 104.14)
+		)
+		(stroke
+			(width 0)
+			(type default)
+		)
+	)
+	(wire
+		(pts
 			(xy 21.59 137.16) (xy 25.4 137.16)
 		)
@@
 		)
 		(stroke
+			(width 0)
+			(type default)
+		)
+	)
+	(wire
+		(pts
+			(xy 105.41 184.15) (xy 187.96 101.6)
+		)
+		(stroke
