File: vanguard/board versions/Vang_V2.3.3/Vanguard_new.kicad_pcb (KiCad board)
At the start: 4 copper layers, 46.4 x 51.9 mm, 93 parts, among them J1 USB_C_Receptacle_USB2.0_16P, J2 Conn_02x03_Pin, J3 Micro_SD_Card_Det1, J4 STARBOARD_SERVO, J5 PORTSIDE_SERVO, J6 Battery In, J7 EJECTION_SERVO, Q1 BSS138, Q2 BSS138, Q3 BSS138, Q4 BSS138, U1 ATSAMD11D14A-M, U10 BMP390L, U2 ATmega4809-A, U3 AT25DF641A-SH-T, U4 AP2112K-3.3, U5 BD1020HFV, U6 BNO086, U7 TXB0104D, U8 TPS61092, U9 MPM3610AGQV-P, Y1 32.768kHz

Commit message: 2.3.3 fix
Parts:
- removed ADR1: ~, Jumper:SolderJumper-2_P1.3mm_Bridged2Bar_Pad1.0x1.5mm
- removed D6: PMEG6020ER, Diode_SMD:Nexperia_CFP3_SOD-123W
- removed L1: 6u8, Inductor_SMD:L_0402_1005Metric
- removed PORTSIDE_RGB1, STARBOARD_RGB1: SMLVN6RGB, LED_SMD:LED_ROHM_SMLVN6
- removed R32: 5k1, Resistor_SMD:R_0402_1005Metric
- removed R33: 5m, Resistor_SMD:R_0402_1005Metric
- removed R36: 4.7kΩ, Resistor_SMD:R_0402_1005Metric
- removed the REF** at (95.5, 87.0)
- removed the REF** at (131.5, 87.0)
- removed the REF** at (131.4, 132.8)
- removed U10: BMP390L, BMP390L:XDCR_BMP390L
- removed U2: ATmega4809-A, Package_QFP:TQFP-48_7x7mm_P0.5mm
- removed U4: AP2112K-3.3, Package_TO_SOT_SMD:SOT-23-5
- added C1: 4n7, Capacitor_SMD:C_0201_0603Metric, F.Cu at (202.6, 175.0)
- added C14: 10uF, Capacitor_SMD:C_0201_0603Metric, F.Cu at (207.5, 175.0)
- added C15: 3.3 nF, Capacitor_SMD:C_0201_0603Metric, F.Cu at (207.5, 176.8)
- added C16: 22uF, Capacitor_SMD:C_0201_0603Metric, F.Cu at (207.5, 178.5)
- added C17: 0.1uF, Capacitor_SMD:C_0201_0603Metric, F.Cu at (207.5, 180.2)
- added C18: 1u, Capacitor_SMD:C_0201_0603Metric, F.Cu at (207.5, 182.0)
- added C19: 0.1uF, Capacitor_SMD:C_0201_0603Metric, F.Cu at (207.5, 183.8)
- added C20: 0.1uF, Capacitor_SMD:C_0201_0603Metric, F.Cu at (210.0, 175.0)
- added C21: 0.1uF, Capacitor_SMD:C_0201_0603Metric, F.Cu at (210.0, 176.8)
- added C22: C, Capacitor_SMD:C_0201_0603Metric, F.Cu at (210.0, 178.5)
- added C23: C, Capacitor_SMD:C_0201_0603Metric, F.Cu at (210.0, 180.2)
- added D12: PMEG6020ER, Diode_SMD:Nexperia_CFP3_SOD-123W, F.Cu at (204.9, 171.5)
- added D13: LED, LED_SMD:LED_0201_0603Metric, F.Cu at (188.3, 187.6)
- added D14: LED, LED_SMD:LED_0201_0603Metric, F.Cu at (188.3, 189.3)
- added D8: SMLVN6RGB, LED_SMD:LED_ROHM_SMLVN6, F.Cu at (214.3, 181.5)
- added R37: 100k, Resistor_SMD:R_0402_1005Metric, F.Cu at (185.4, 194.4)
- added R38: 100, Resistor_SMD:R_0402_1005Metric, F.Cu at (185.4, 196.4)
- added R39: 330, Resistor_SMD:R_0402_1005Metric, F.Cu at (185.4, 198.4)
- added REF**: MountingHole_2.1mm, MountingHole:MountingHole_2.1mm, F.Cu at (293.8, 161.1)
- added TP8: TestPoint, TestPoint:TestPoint_Pad_1.0x1.0mm, F.Cu at (211.0, 198.2)
- added TP9: TestPoint, TestPoint:TestPoint_Pad_1.0x1.0mm, F.Cu at (211.0, 201.2)
- added U12: AP2112K-3.3, Package_TO_SOT_SMD:SOT-23-5, F.Cu at (212.6, 171.4)
- C10: value 100u -> 1uF; footprint Capacitor_SMD:CP_Elec_6.3x5.4 -> Capacitor_SMD:C_0201_0603Metric
- C11: value 1u -> 100nF
- C12: value 4n7 -> 2u2
- C13: value 100n -> 100u; footprint Capacitor_SMD:C_0201_0603Metric -> Capacitor_SMD:CP_Elec_6.3x5.4
- C2: value 22p -> 100n
- C3: value 22p -> 0.1uF
- C4: value 22u -> 22pF
- C5: value 22u -> 22p
- C6: value 1u -> 0.1uF
- C7: value 0u1 -> 0.1uF
- C9: value 2u2 -> C
- D1: value PRTR5V0U2X -> LED; footprint Package_TO_SOT_SMD:SOT-143 -> LED_SMD:LED_0201_0603Metric
- D2: value LED -> PRTR5V0U2X; footprint LED_SMD:LED_0201_0603Metric -> Package_TO_SOT_SMD:SOT-143
- D5: value GREEN -> LED
- D7: value LED -> SMLVN6RGB; footprint LED_SMD:LED_0201_0603Metric -> LED_SMD:LED_ROHM_SMLVN6
- J1: footprint Connector_USB:USB-C-SMD_JLC REPLACEMENT -> Connector_USB:USB_C_Receptacle_Amphenol_124019772112A
- J2: value Conn_02x03_Pin -> Micro_SD_Card_Det1; footprint Connector_PinHeader_2.54mm:PinHeader_2x03_P2.54mm_Vertical -> Connector_Card:microSD_HC_Hirose_DM3D-SF
- J3: value Micro_SD_Card_Det1 -> Conn_02x03_Odd_Even; footprint Connector_Card:microSD_HC_Hirose_DM3D-SF -> Connector_PinHeader_2.54mm:PinHeader_2x03_P2.54mm_Vertical
- J4: value STARBOARD_SERVO -> Conn_01x03
- J5: value PORTSIDE_SERVO -> Conn_01x03
- J6: value Battery In -> Conn_01x03; footprint Connector_JST:JST_PH_B2B-PH-K_1x02_P2.00mm_Vertical -> Connector_PinHeader_2.54mm:PinHeader_1x03_P2.54mm_Vertical
- J7: value EJECTION_SERVO -> Conn_01x02_Pin; footprint Connector_PinHeader_2.54mm:PinHeader_1x03_P2.54mm_Vertical -> Connector_JST:JST_PH_B2B-PH-K_1x02_P2.00mm_Vertical
- R1: value 4.7kΩ -> 2k2
- R11, R13: value 4k7 -> 330
- R12: value 4k7 -> 0
- R14: value 100k -> 4k7
- R15: value 100k -> R
- R16: value 19k1 -> 4k7
- R17: value 330R -> 4k7
- R18: value 10k -> 4k7
- R2: value 4k7 -> 2k2
- R21, R22: value 2k2 -> 220
- R23, R24: value 10k -> 220
- R27, R28, R30: value 220 -> 100k
- R29: value 220 -> 315k
- R3: value 330 -> 10k
- R31: value 5k1 -> 10k
- R35: value R220 -> 124k
- R5: value 0 -> 5k1
- R6: value 4k7 -> 5k1
- R8: value DNP -> 4k7
- U1: value ATSAMD11D14A-M -> TXB0104D; footprint Package_DFN_QFN:QFN-24-1EP_4x4mm_P0.5mm_EP2.6x2.6mm -> Package_SO:SOIC-14_3.9x8.7mm_P1.27mm
- U3: value AT25DF641A-SH-T -> ATSAMD11D14A-M; footprint Package_SO:SOIC-8_3.9x4.9mm_P1.27mm -> Package_DFN_QFN:QFN-24-1EP_4x4mm_P0.5mm_EP2.6x2.6mm
- U5: value BD1020HFV -> BD1020HFV-TR
- U6: value BNO086 -> AT25DF641A-SH-T; footprint Package_LGA:LGA-28_5.2x3.8mm_P0.5mm -> Package_SO:SOIC-8_3.9x4.9mm_P1.27mm
- U7: value TXB0104D -> ATmega4809-A; footprint Package_SO:SOIC-14_3.9x8.7mm_P1.27mm -> Package_QFP:TQFP-48_7x7mm_P0.5mm
- U8: value TPS61092 -> BNO055; footprint Package_DFN_QFN:DFN-10-1EP_3x3mm_P0.5mm_EP1.65x2.38mm_ThermalVias -> Package_LGA:LGA-28_5.2x3.8mm_P0.5mm
- U9: value MPM3610AGQV-P -> TPS61092; footprint Package_DFN_QFN:QFN-20-1EP_4x4mm_P0.5mm_EP2.5x2.5mm_ThermalVias -> Package_DFN_QFN:Texas_RSA_VQFN-16-1EP_4x4mm_P0.65mm_EP2.7x2.7mm_ThermalVias
- Y1: value 32.768kHz -> Crystal
- moved C13 145.5 mm to (208.7, 189.6), turned to 0 degrees
- moved J6 141.6 mm to (186.8, 201.7), turned to 0 degrees
- moved D2 140.8 mm to (197.1, 206.4), turned to 0 degrees
- moved J5 138.7 mm to (182.2, 201.7)
- moved C12 138.5 mm to (205.1, 183.8), turned to 0 degrees
- moved J4 138.2 mm to (177.5, 201.7)
- moved TP6 134.1 mm to (208.0, 201.2), turned to 0 degrees
- moved J3 133.9 mm to (214.9, 195.9), turned to 0 degrees
- moved C8 133.9 mm to (205.1, 176.8), turned to 0 degrees
- moved TP3 132.5 mm to (204.9, 201.2), turned to 0 degrees
- moved U8 132.4 mm to (213.6, 166.2), turned to 0 degrees
- moved C10 131.5 mm to (205.1, 180.2), turned to 0 degrees
- moved TP7 131.4 mm to (211.0, 195.2)
- moved Q3 130.6 mm to (192.5, 197.1), turned to 0 degrees
- moved TP5 130.3 mm to (208.0, 198.2)
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Connections:
- BZ1 pad 1: Net-(BZ1-+) -> +3.3V
- BZ1 pad 2: GND -> Net-(BZ1--)
- C10 pad 1: +5V -> Net-(U12-EN)
- C11 pad 1: Net-(D6-K) -> GND
- C11 pad 2: GND -> +3.3V
- C12 pad 1: BATT_IN -> +5V
- C13 pad 1: BATT_IN -> +5V
- C2 pad 1: Net-(U6-XOUT32/CLKSEL1) -> GND
- C2 pad 2: GND -> VBUS
- C3 pad 1: Net-(U6-XIN32) -> Net-(U8-CAP)
- C4 pad 1: Net-(U9-IN) -> Net-(U8-XOUT32)
- C5 pad 1: Net-(D6-K) -> Net-(U8-XIN32)
- C7 pad 1: Net-(U6-CAP) -> GND
- C7 pad 2: GND -> +3.3V
- C8 pad 1: BATT_IN -> Net-(J7-Pin_1)
- C9 pad 1: +5V -> GND
- C9 pad 2: GND -> +3.3V
- D1 pad 2: Net-(D1-I/O1) -> Net-(D1-A)
- D2 pad 1: Net-(D2-K) -> GND
- D2 pad 2: Net-(D2-A) -> Net-(D2-I/O1)
- D5 pad 1: GND -> Net-(D5-K)
- D7 pad 1: BATT_IN -> Net-(D7-BA)
- D7 pad 2: Net-(D7-A) -> Net-(D7-RA)
- J1 pad A4: BATT_IN -> VBUS
- J1 pad A6: Net-(D1-I/O1) -> Net-(D2-I/O1)
- J1 pad A7: Net-(D1-I/O2) -> Net-(D2-I/O2)
- J1 pad A9: BATT_IN -> VBUS
- J1 pad B4: BATT_IN -> VBUS
- J1 pad B6: Net-(D1-I/O1) -> Net-(D2-I/O1)
- J1 pad B7: Net-(D1-I/O2) -> Net-(D2-I/O2)
- J1 pad B9: BATT_IN -> VBUS
- J2 pad 1: +3.3V -> unconnected-(J2-DAT2-Pad1)
- J2 pad 2: Net-(J2-Pin_2) -> unconnected-(J2-DAT3/CD-Pad2)
- J2 pad 3: Net-(J2-Pin_3) -> Net-(J2-CMD)
- J2 pad 4: UPDI -> +3.3V
- J2 pad 5: GND -> Net-(J2-CLK)
- J2 pad 6: Net-(J2-Pin_6) -> +3.3V
- J3 pad 1: unconnected-(J3-DAT2-Pad1) -> +3.3V
- J3 pad 2: unconnected-(J3-DAT3/CD-Pad2) -> Net-(J3-Pin_2)
- J3 pad 3: Net-(J3-CMD) -> Net-(J3-Pin_3)
- J3 pad 4: GND -> UPDI
- J3 pad 5: Net-(J3-CLK) -> GND
- J3 pad 6: +3.3V -> Net-(J3-Pin_6)
- J4 pad 1: STAR_SERVO -> PORT_SERVO
- J5 pad 1: PORT_SERVO -> STAR_SERVO
- J6 pad 1: BATT_IN -> EJEC_SERVO
- J6 pad 2: GND -> +5V
- J7 pad 1: EJEC_SERVO -> Net-(J7-Pin_1)
- J7 pad 2: +5V -> GND
- JP1 pad 2: GND -> +3.3V
- JP2 pad 2: +3.3V -> GND
- Q2 pad 2: Net-(D3-K) -> Net-(D5-K)
- Q3 pad 2: Net-(D2-K) -> Net-(D3-K)
- Q4 pad 3: Net-(BZ1-+) -> Net-(BZ1--)
- R1 pad 2: SCL -> SDA
- R10 pad 2: Net-(D3-K) -> SCL
- R11 pad 2: Net-(J2-Pin_6) -> Net-(D3-A)
- R12 pad 1: +3.3V -> /RX_UPDI
- R12 pad 2: RX0 -> /TX_UPDI
- R13 pad 2: TX0 -> Net-(D5-A)
- R14 pad 1: Net-(U9-IN) -> +3.3V
- R14 pad 2: Net-(U9-EN) -> /TX_UPDI
- R15 pad 1: Net-(D6-K) -> /TX_UPDI
- R15 pad 2: Net-(U9-FB) -> UPDI
- R16 pad 1: Net-(U9-FB) -> +3.3V
- R16 pad 2: GND -> UPDI
- R17 pad 2: Net-(D5-A) -> Net-(D5-K)
- R18 pad 1: Net-(U6-~{RST}) -> +3.3V
- R18 pad 2: +3.3V -> TX0
- R19 pad 1: Net-(U6-ENV_SCL) -> +3.3V
- R19 pad 2: +3.3V -> Net-(D3-K)
- R2 pad 2: Net-(J2-Pin_3) -> SCL
- R20 pad 1: Net-(U6-ENV_SDA) -> +3.3V
- R20 pad 2: +3.3V -> RX0
- R21 pad 1: +3.3V -> STAR_BLUE
- R21 pad 2: SDA -> Net-(D7-BA)
- R22 pad 1: +3.3V -> STAR_RED
- R22 pad 2: SCL -> Net-(D7-RA)
- R23 pad 1: +3.3V -> STAR_GREEN
- R23 pad 2: Net-(ADR1-B) -> Net-(D7-GA)
- R24 pad 1: +3.3V -> Net-(D8-BA)
- R24 pad 2: Net-(U6-~{BOOT}) -> PORT_BLUE
- R25 pad 1: STAR_BLUE -> Net-(D8-RA)
- R25 pad 2: Net-(STARBOARD_RGB1-BA) -> PORT_RED
- R26 pad 1: STAR_RED -> Net-(D8-GA)
- R26 pad 2: Net-(STARBOARD_RGB1-RA) -> PORT_GREEN
- R27 pad 1: STAR_GREEN -> Net-(J7-Pin_1)
- R27 pad 2: Net-(STARBOARD_RGB1-GA) -> Net-(U9-LBI)
- R28 pad 1: Net-(PORTSIDE_RGB1-BA) -> Net-(U9-LBI)
- R28 pad 2: PORT_BLUE -> GND
- R29 pad 1: Net-(PORTSIDE_RGB1-RA) -> +5V
- R29 pad 2: PORT_RED -> Net-(U9-FB)
- R3 pad 1: +3.3V -> Net-(U8-~{RESET})
- R3 pad 2: Net-(D3-A) -> +3.3V
- R30 pad 1: Net-(PORTSIDE_RGB1-GA) -> Net-(U9-FB)
- R30 pad 2: PORT_GREEN -> GND
- R31 pad 1: Net-(J1-CC1) -> +3.3V
- R31 pad 2: GND -> PA3/SS
- R35 pad 1: Net-(D7-A) -> Net-(U12-EN)
- R35 pad 2: BATT_IN -> Net-(U11-FB)
- R4 pad 1: +3.3V -> Net-(D1-A)
- R4 pad 2: Net-(D2-A) -> VBUS
- R5 pad 1: /RX_UPDI -> Net-(J1-CC1)
- R5 pad 2: /TX_UPDI -> GND
- R6 pad 1: +3.3V -> Net-(J1-CC2)
- R6 pad 2: /TX_UPDI -> GND
- R7 pad 2: UPDI -> SDA
- R8 pad 1: /TX_UPDI -> +3.3V
- R8 pad 2: UPDI -> Net-(J3-Pin_6)
- R9 pad 2: Net-(D2-K) -> Net-(J3-Pin_3)
- TP1 pad 1: Net-(D1-I/O1) -> D4
- TP2 pad 1: Net-(D1-I/O2) -> SCL
- TP3 pad 1: D4 -> Net-(D2-I/O1)
- TP4 pad 1: PA2/SCK -> Net-(D2-I/O2)
- TP5 pad 1: Net-(U6-XIN32) -> Net-(U8-XOUT32)
- TP6 pad 1: Net-(U6-XOUT32/CLKSEL1) -> PA2/SCK
- TP7 pad 1: SCL -> Net-(U8-~{BOOT_LOAD_PIN})
- U1 pad 1: unconnected-(U1-PA02-Pad1) -> +3.3V
- U1 pad 10: unconnected-(U1-PA11-Pad10) -> D5
- U1 pad 11: /TX_UPDI -> D4
- U1 pad 12: /RX_UPDI -> D6
- U1 pad 13: unconnected-(U1-PA16-Pad13) -> D7
- U1 pad 14: unconnected-(U1-PA17-Pad14) -> +3.3V
- U1 pad 2: unconnected-(U1-PA03-Pad2) -> Net-(J2-DAT1)
- U1 pad 3: unconnected-(U1-PA04-Pad3) -> Net-(J2-DAT0)
- U1 pad 4: unconnected-(U1-PA05-Pad4) -> Net-(J2-CLK)
- U1 pad 5: unconnected-(U1-PA06-Pad5) -> Net-(J2-CMD)
- U1 pad 7: unconnected-(U1-PA08/XIN-Pad7) -> GND
- U1 pad 8: unconnected-(U1-PA09/XOUT-Pad8) -> +3.3V
- U3 pad 1: PA3/SS -> unconnected-(U3-PA02-Pad1)
- U3 pad 2: PA0/MISO -> unconnected-(U3-PA03-Pad2)
- U3 pad 3: WP -> unconnected-(U3-PA04-Pad3)
- U3 pad 4: GND -> unconnected-(U3-PA05-Pad4)
- U3 pad 5: PA1/MOSI -> unconnected-(U3-PA06-Pad5)
- U3 pad 6: PA2/SCK -> unconnected-(U3-PA07-Pad6)
- U3 pad 7: HOLD -> unconnected-(U3-PA08/XIN-Pad7)
- U3 pad 8: +3.3V -> unconnected-(U3-PA09/XOUT-Pad8)
- U6 pad 1: unconnected-(U6-RESV_NC-Pad1) -> PA3/SS
- U6 pad 2: GND -> PA0/MISO
- U6 pad 3: +3.3V -> WP
- U6 pad 4: Net-(U6-~{BOOT}) -> GND
- U6 pad 5: PS1 -> PA1/MOSI
- U6 pad 6: PS0/WAKE -> PA2/SCK
- U6 pad 7: unconnected-(U6-RESV_NC-Pad7) -> HOLD
- U6 pad 8: unconnected-(U6-RESV_NC-Pad8) -> +3.3V
- U7 pad 1: +3.3V -> PA2/SCK
- U7 pad 10: D5 -> STAR_RED
- U7 pad 11: D4 -> STAR_GREEN
- U7 pad 12: D6 -> SDA
- U7 pad 13: D7 -> PORT_SERVO
- U7 pad 2: Net-(J3-DAT1) -> PA1/MOSI
- U7 pad 3: Net-(J3-DAT0) -> PA0/MISO
- U7 pad 4: Net-(J3-CLK) -> unconnected-(U7-PB0-Pad4)
- U7 pad 5: Net-(J3-CMD) -> unconnected-(U7-PB1-Pad5)
- U7 pad 6: unconnected-(U7-NC-Pad6) -> STAR_BLUE
- U7 pad 7: GND -> unconnected-(U7-PB3-Pad7)
- U7 pad 8: +3.3V -> TX0
- U7 pad 9: unconnected-(U7-NC-Pad9) -> RX0
- U8 pad 1: +5V -> unconnected-(U8-PIN1-Pad1)
- U8 pad 10: GND -> unconnected-(U8-BL_IND-Pad10)
- U8 pad 11: BATT_IN -> Net-(U8-~{RESET})
- U8 pad 2: unconnected-(U8-NC-Pad2) -> GND
- U8 pad 3: GND -> +3.3V
- U8 pad 4: Net-(L1-Pad2) -> Net-(U8-~{BOOT_LOAD_PIN})
- U8 pad 7: GND -> unconnected-(U8-PIN7-Pad7)
- U8 pad 8: BATT_IN -> unconnected-(U8-PIN8-Pad8)
- U8 pad 9: unconnected-(U8-LBI-Pad9) -> Net-(U8-CAP)
- U9 pad 1: Net-(U9-FB) -> +5V
- U9 pad 10: (no net) -> GND
- U9 pad 11: unconnected-(U9-BST-Pad11) -> Net-(J7-Pin_1)
- U9 pad 12: GND -> unconnected-(U9-LBO-Pad12)
- U9 pad 14: GND -> Net-(U9-FB)
- U9 pad 15: (no net) -> +5V
- U9 pad 16: Net-(U9-IN) -> +5V
- U9 pad 17: Net-(U9-EN) -> GND
- U9 pad 3: GND -> Net-(L1-Pad2)
- U9 pad 4: unconnected-(U9-SW-Pad19)_2 -> Net-(L1-Pad2)
- U9 pad 5: unconnected-(U9-SW-Pad19)_3 -> GND
- U9 pad 6: unconnected-(U9-SW-Pad19)_1 -> GND
- U9 pad 7: Net-(D6-K) -> GND
- U9 pad 8: Net-(D6-K) -> Net-(J7-Pin_1)
- U9 pad 9: Net-(D6-K) -> Net-(U9-LBI)
- Y1 pad 1: Net-(U6-XOUT32/CLKSEL1) -> Net-(U8-XIN32)
- Y1 pad 2: Net-(U6-XIN32) -> Net-(U8-XOUT32)
Routing:
- net +3.3V: track 201.1 -> 0.00 mm, vias 27 -> 0
- net BATT_IN: track 97.9 -> 0.00 mm, vias 3 -> 0
- net GND: track 76.5 -> 0.00 mm, vias 41 -> 0
- net CD: track 69.4 -> 0.00 mm, vias 2 -> 0
- net UPDI: track 50.5 -> 0.00 mm, vias 2 -> 0
- net EJEC_SERVO: track 47.2 -> 0.00 mm, vias 1 -> 0
- net +5V: track 40.2 -> 0.00 mm, vias 2 -> 0
- net PORT_SERVO: track 39.2 -> 0.00 mm, vias 1 -> 0
- net RX0: track 37.6 -> 0.00 mm, vias 2 -> 0
- net D4: track 35.8 -> 0.00 mm, vias 4 -> 0
- net STAR_SERVO: track 33.1 -> 0.00 mm, vias 1 -> 0
- net BUZZER: track 32.4 -> 0.00 mm, vias 2 -> 0
- net D5: track 31.0 -> 0.00 mm, vias 2 -> 0
- net D7: track 30.8 -> 0.00 mm
- net Net-(D6-K): track 30.8 -> 0.00 mm, vias 2 -> 0
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- removed copper zone on In1.Cu, net GND
- removed copper zone on In2.Cu, net GND
Other:
- board size 46.4 x 51.9 mm -> 42.3 x 51.9 mm

Commit message: finished input usb
Parts:
- removed C23, C9: C, Capacitor_SMD:C_0201_0603Metric
- removed Q1, Q2, Q3: BSS138, Package_TO_SOT_SMD:SOT-23
- removed R14, R16, R17, R18, R19, R20: 4k7, Resistor_SMD:R_0402_1005Metric
- removed R15: R, Resistor_SMD:R_0402_1005Metric
- removed U7: ATmega4809-A, Package_QFP:TQFP-48_7x7mm_P0.5mm
- added C26: 0.1uF, Capacitor_SMD:C_0603_1608Metric, F.Cu at (209.3, 171.3)
- added C27: 0.1uF, Capacitor_SMD:C_0603_1608Metric, F.Cu at (209.3, 173.8)
- added L1: SLF7055T-6R8N2R8-3PF, Package_LGA:ST_HLGA-10_2x2mm_P0.5mm_LayoutBorder3x2y, F.Cu at (225.1, 182.5)
- added R32: 10k, Resistor_SMD:R_0603_1608Metric, F.Cu at (221.3, 168.8)
- added R33: 10k, Resistor_SMD:R_0603_1608Metric, F.Cu at (221.3, 171.3)
- added U10: ATmega4809-A, Package_QFP:TQFP-48_7x7mm_P0.5mm, F.Cu at (204.9, 190.8)
- added U4: BMP390L, Package_LGA:ST_HLGA-10_2x2mm_P0.5mm_LayoutBorder3x2y, F.Cu at (228.7, 182.5)
- C1, C10, C11, C12, C14, C15, C16, C17, C18, C19, C2, C20, C21, C22, C3, C4, C5, C6, C7, C8: footprint Capacitor_SMD:C_0201_0603Metric -> Capacitor_SMD:C_0603_1608Metric
- C13: footprint Capacitor_SMD:CP_Elec_6.3x5.4 -> Capacitor_SMD:C_0603_1608Metric
- R1, R10, R11, R12, R13, R2, R21, R22, R23, R24, R25, R26, R27, R28, R29, R3, R30, R31, R34, R37, R38, R39, R4, R5, R6, R7, R8, R9: footprint Resistor_SMD:R_0402_1005Metric -> Resistor_SMD:R_0603_1608Metric
- R35: value 124k -> 350; footprint Resistor_SMD:R_0402_1005Metric -> Resistor_SMD:R_0603_1608Metric
- U1: value TXB0104D -> TPS82130; footprint Package_SO:SOIC-14_3.9x8.7mm_P1.27mm -> Package_LGA:Texas_SIL0008D_MicroSiP-8-1EP_2.8x3mm_P0.65mm_EP1.1x1.9mm_ThermalVias
- moved J1 185.9 mm to (333.1, 294.3), turned to 90 degrees
- moved R5 182.9 mm to (326.6, 295.1), turned to 180 degrees
- moved R6 180.7 mm to (326.6, 293.3), turned to 180 degrees
- moved R4 179.5 mm to (324.4, 290.4), turned to -90 degrees
- moved R11 179.3 mm to (316.6, 300.1), turned to 90 degrees
- moved R13 175.4 mm to (314.9, 300.0), turned to 90 degrees
- moved R9 174.6 mm to (319.8, 298.4), turned to 90 degrees
- moved R8 174.5 mm to (318.2, 298.4), turned to 90 degrees
- moved R12 172.8 mm to (313.7, 295.4), turned to 90 degrees
- moved D1 172.5 mm to (324.3, 288.5)
- moved D3 171.5 mm to (316.7, 297.8), turned to -90 degrees
- moved C1 170.0 mm to (327.4, 290.4), turned to -90 degrees
- moved D5 169.0 mm to (314.9, 297.8), turned to -90 degrees
- moved C2 167.6 mm to (325.9, 290.4), turned to -90 degrees
- moved J3 161.5 mm to (332.4, 306.8), turned to 180 degrees
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Connections:
- net PA3/SS renamed FLASH_CS
- C15 pad 1: Net-(U11-SS/TR) -> Net-(U1-SS/TR)
- D3 pad 1: Net-(D3-K) -> TX0
- D5 pad 1: Net-(D5-K) -> RX0
- J1 pad S1: unconnected-(J1-SHIELD-PadS1)_2 -> GND
- J2 pad 2: unconnected-(J2-DAT3/CD-Pad2) -> SD_CS
- J2 pad 3: Net-(J2-CMD) -> MOSI
- J2 pad 5: Net-(J2-CLK) -> SCK
- J2 pad 6: +3.3V -> GND
- J2 pad 7: Net-(J2-DAT0) -> MISO
- J2 pad 8: Net-(J2-DAT1) -> unconnected-(J2-DAT1-Pad8)
- R12 pad 2: /TX_UPDI -> UPDI
- R35 pad 2: Net-(U11-FB) -> Net-(U1-FB)
- R37 pad 1: Net-(U11-FB) -> Net-(U1-FB)
- TP1 pad 1: D4 -> SCK
- TP6 pad 1: PA2/SCK -> SCK
- U1 pad 1: +3.3V -> Net-(D12-K)
- U1 pad 2: Net-(J2-DAT1) -> Net-(D12-K)
- U1 pad 3: Net-(J2-DAT0) -> GND
- U1 pad 4: Net-(J2-CLK) -> Net-(U12-EN)
- U1 pad 5: Net-(J2-CMD) -> Net-(U12-EN)
- U1 pad 6: unconnected-(U1-NC-Pad6) -> Net-(U1-FB)
- U1 pad 7: GND -> unconnected-(U1-PG-Pad7)
- U1 pad 8: +3.3V -> Net-(U1-SS/TR)
- U1 pad 9: unconnected-(U1-NC-Pad9) -> GND
- U3 pad 11: /TX_UPDI -> UPDI
- U3 pad 15: Net-(D3-K) -> RX0
- U3 pad 16: Net-(D5-K) -> TX0
- U6 pad 2: PA0/MISO -> MISO
- U6 pad 5: PA1/MOSI -> MOSI
- U6 pad 6: PA2/SCK -> SCK
Routing:
- net Net-(J3-Pin_3): track 0.00 -> 18.9 mm
- net GND: track 0.00 -> 18.8 mm, vias 0 -> 8
- net VBUS: track 0.00 -> 18.4 mm
- net Net-(J3-Pin_2): track 0.00 -> 17.8 mm, vias 0 -> 1
- net Net-(D2-I/O1): track 0.00 -> 15.1 mm
- net Net-(J3-Pin_6): track 0.00 -> 15.0 mm, vias 0 -> 2
- net Net-(D2-I/O2): track 0.00 -> 14.6 mm, vias 0 -> 2
- net Net-(J1-CC2): track 0.00 -> 5.46 mm, vias 0 -> 2
- net RX0: track 0.00 -> 2.78 mm
- net Net-(J1-CC1): track 0.00 -> 2.48 mm
- net +3.3V: track 0.00 -> 2.29 mm
- net /RX_UPDI: track 0.00 -> 1.84 mm
- net UPDI: track 0.00 -> 1.69 mm
- net TX0: track 0.00 -> 1.59 mm
- net Net-(D1-A): track 0.00 -> 1.19 mm
- added copper zone on B.Cu, net (none)
- added copper zone on F.Cu, net (none)
- added copper zone on In1.Cu, net GND
- added copper zone on In2.Cu, net GND
Other:
- board size 42.3 x 51.9 mm -> 100 x 241.7 mm

Commit message: started pcb
Parts:
- removed REF**: MountingHole_2.1mm, MountingHole:MountingHole_2.1mm
- C1, C2, D1, D2, J1, J2, R4, U1, U10, U12, U3, U4, U6, U8, U9: moved to B.Cu
- C26, C27: footprint Capacitor_SMD:C_0603_1608Metric -> Capacitor_SMD:C_0201_0603Metric
- R32, R33: footprint Resistor_SMD:R_0603_1608Metric -> Resistor_SMD:R_0201_0603Metric
- moved R12 344.0 mm to (83.5, 39.8), turned to 0 degrees
- moved J3 343.3 mm to (141.5, 21.4), turned to 90 degrees
- moved R13 341.6 mm to (91.9, 41.2), turned to 0 degrees
- moved C11 340.6 mm to (71.5, 57.4), turned to 0 degrees
- moved D5 338.4 mm to (94.2, 41.2), turned to 180 degrees
- moved R11 335.4 mm to (115.5, 31.7), turned to 0 degrees
- moved D3 332.1 mm to (117.8, 31.8), turned to 180 degrees
- moved R8 331.5 mm to (127.6, 27.2), turned to -90 degrees
- moved R9 331.4 mm to (129.6, 27.1), turned to -90 degrees
- moved R5 327.4 mm to (138.3, 27.2), turned to 90 degrees
- moved R4 325.7 mm to (134.9, 25.4)
- moved J1 325.6 mm to (143.7, 29.4), turned to -90 degrees
- moved D2 325.3 mm to (133.8, 29.0), turned to 135 degrees
- moved C2 325.2 mm to (136.4, 26.1)
- moved C1 325.2 mm to (138.0, 26.1)
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Routing:
- net UPDI: track 1.69 -> 31.6 mm
- net Net-(J3-Pin_6): track 15.0 -> 27.7 mm, vias 2 -> 1
- net Net-(J3-Pin_3): track 18.9 -> 25.9 mm, vias 0 -> 1
- net Net-(D12-K): track 0.00 -> 6.47 mm, vias 0 -> 1
- net Net-(D1-A): track 1.19 -> 4.71 mm
- net GND: track 18.8 -> 15.7 mm, vias 8 -> 10
- net RX0: track 2.78 -> 0.00 mm
- net +3.3V: track 2.29 -> 0.00 mm
- net /RX_UPDI: track 1.84 -> 0.00 mm
- net TX0: track 1.59 -> 0.00 mm
- net Net-(D2-I/O2): track 14.6 -> 16.0 mm
- net Net-(J3-Pin_2): track 17.8 -> 16.6 mm
- net VBUS: track 18.4 -> 19.6 mm
- net Net-(J1-CC2): track 5.46 -> 5.06 mm, vias 2 -> 1
- net Net-(D2-I/O1): track 15.1 -> 14.8 mm, vias 0 -> 2
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Other:
- board size 100 x 241.7 mm -> 276.7 x 289.9 mm

Commit message: dont touch yet
Parts:
- added REF**: C_0201_0603Metric, Capacitor_SMD:C_0201_0603Metric, F.Cu at (173.9, 128.5)
- C8, J7, Q4, R27: moved to B.Cu
- L1: footprint Package_LGA:ST_HLGA-10_2x2mm_P0.5mm_LayoutBorder3x2y -> Inductor_SMD:L_7.3x7.3_H4.5
- moved C7 152.0 mm to (186.4, 137.1)
- moved D13 143.1 mm to (155.5, 128.6)
- moved TP1 141.9 mm to (191.1, 137.6), turned to 90 degrees
- moved U1 137.2 mm to (150.2, 124.7), turned to 180 degrees
- moved D14 134.2 mm to (156.9, 119.4), turned to 90 degrees
- moved C5 133.5 mm to (174.3, 116.4), turned to -90 degrees
- moved C14 133.4 mm to (150.0, 122.0), turned to 180 degrees
- moved C3 133.2 mm to (172.1, 122.5), turned to -90 degrees
- moved C4 128.8 mm to (169.2, 116.5), turned to -90 degrees
- moved D12 128.7 mm to (151.9, 118.9), turned to 90 degrees
- moved C19 127.5 mm to (172.3, 119.0), turned to 90 degrees
- moved C17 125.4 mm to (170.7, 119.1), turned to -90 degrees
- moved R3 123.4 mm to (170.5, 122.5), turned to -90 degrees
- moved R37 121.8 mm to (150.3, 127.5), turned to 180 degrees
- moved R35 121.6 mm to (152.7, 126.7), turned to -90 degrees
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- renumbered C19 to C17, C17 to C19
Routing:
- net +3.3V: track 0.00 -> 231.4 mm, vias 0 -> 24
- net GND: track 15.7 -> 75.7 mm, vias 10 -> 50
- net SDA: track 0.00 -> 59.1 mm, vias 0 -> 5
- net STAR_GREEN: track 0.00 -> 53.9 mm, vias 0 -> 3
- net STAR_RED: track 0.00 -> 53.1 mm, vias 0 -> 3
- net SCL: track 0.00 -> 50.9 mm, vias 0 -> 5
- net STAR_BLUE: track 0.00 -> 38.3 mm, vias 0 -> 1
- net MISO: track 0.00 -> 36.3 mm, vias 0 -> 2
- net SCK: track 0.00 -> 35.0 mm, vias 0 -> 4
- net RX0: track 0.00 -> 34.2 mm, vias 0 -> 2
- net STAR_SERVO: track 0.00 -> 33.2 mm, vias 0 -> 2
- net WP: track 0.00 -> 33.0 mm, vias 0 -> 3
- net TEMP_SENSOR: track 0.00 -> 30.7 mm, vias 0 -> 1
- net +5V: track 0.00 -> 30.7 mm, vias 0 -> 3
- net PORT_BLUE: track 0.00 -> 29.7 mm, vias 0 -> 3
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Other:
- board size 276.7 x 289.9 mm -> 57.6 x 40 mm

Commit message: save spot
Parts:
- removed REF**: C_0201_0603Metric, Capacitor_SMD:C_0201_0603Metric
- J7, Q4: moved to F.Cu
- moved R33 181.8 mm to (184.1, 306.5), turned to -45 degrees
- moved R32 181.2 mm to (183.4, 306.8), turned to -45 degrees
- moved U10 181.0 mm to (179.6, 310.9), turned to 45 degrees
- moved C27 180.5 mm to (181.0, 312.6), turned to -135 degrees
- moved C26 179.8 mm to (180.4, 308.6), turned to 135 degrees
- moved C1 162.9 mm to (181.0, 267.9)
- moved C11 162.9 mm to (188.0, 274.0)
- moved C19 162.9 mm to (198.6, 279.8)
- moved C5 162.9 mm to (200.6, 277.2)
- moved R1 162.9 mm to (193.6, 275.2)
- moved R12 162.9 mm to (188.2, 281.1)
- moved R3 162.9 mm to (196.8, 283.3)
- moved R4 162.9 mm to (180.4, 271.0)
- moved R5 162.9 mm to (182.2, 267.6)
- moved R6 162.9 mm to (186.9, 267.6)
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Routing:
- net +3.3V: track 231.4 -> 27.5 mm, vias 24 -> 11
- net STAR_GREEN: track 53.9 -> 0.00 mm, vias 3 -> 0
- net STAR_RED: track 53.1 -> 0.00 mm, vias 3 -> 0
- net SDA: track 59.1 -> 7.31 mm, vias 5 -> 2
- net SCL: track 50.9 -> 7.48 mm, vias 5 -> 2
- net STAR_BLUE: track 38.3 -> 0.00 mm, vias 1 -> 0
- net MISO: track 36.3 -> 0.00 mm, vias 2 -> 0
- net STAR_SERVO: track 33.2 -> 0.00 mm, vias 2 -> 0
- net RX0: track 34.2 -> 2.93 mm, vias 2 -> 1
- net TEMP_SENSOR: track 30.7 -> 0.00 mm, vias 1 -> 0
- net WP: track 33.0 -> 2.93 mm, vias 3 -> 1
- net PORT_BLUE: track 29.7 -> 0.00 mm, vias 3 -> 0
- net SCK: track 35.0 -> 6.47 mm, vias 4 -> 1
- net CD: track 28.3 -> 0.00 mm, vias 2 -> 0
- net PORT_SERVO: track 28.0 -> 0.00 mm, vias 1 -> 0
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Other:
- board size 57.6 x 40 mm -> 276.7 x 289.9 mm

Commit message: wiring done
Parts:
- J7, Q4: moved to B.Cu
- moved R33 181.8 mm to (168.1, 125.4), turned to 45 degrees
- moved R32 181.2 mm to (168.4, 126.2), turned to 45 degrees
- moved U10 181.0 mm to (172.5, 130.0), turned to 135 degrees
- moved C27 180.5 mm to (171.8, 132.4), turned to 135 degrees
- moved C26 179.8 mm to (170.2, 129.2), turned to -135 degrees
- moved C1 162.9 mm to (154.7, 107.2)
- moved C11 162.9 mm to (161.7, 113.2)
- moved C19 162.9 mm to (172.3, 119.0)
- moved C5 162.9 mm to (174.3, 116.4)
- moved R1 162.9 mm to (167.3, 114.4)
- moved R12 162.9 mm to (161.9, 120.4)
- moved R3 162.9 mm to (170.5, 122.5)
- moved R4 162.9 mm to (154.1, 110.2)
- moved R5 162.9 mm to (155.9, 106.8)
- moved R6 162.9 mm to (160.6, 106.8)
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Routing:
- net +3.3V: track 27.5 -> 267.5 mm, vias 11 -> 28
- net STAR_GREEN: track 0.00 -> 54.6 mm, vias 0 -> 3
- net STAR_RED: track 0.00 -> 53.1 mm, vias 0 -> 3
- net SDA: track 7.31 -> 59.1 mm, vias 2 -> 5
- net SCL: track 7.48 -> 50.9 mm, vias 2 -> 5
- net STAR_BLUE: track 0.00 -> 38.3 mm, vias 0 -> 1
- net MISO: track 0.00 -> 36.3 mm, vias 0 -> 2
- net STAR_SERVO: track 0.00 -> 33.2 mm, vias 0 -> 2
- net RX0: track 2.93 -> 34.2 mm, vias 1 -> 2
- net TEMP_SENSOR: track 0.00 -> 30.7 mm, vias 0 -> 1
- net WP: track 2.93 -> 33.0 mm, vias 1 -> 3
- net PORT_BLUE: track 0.00 -> 29.7 mm, vias 0 -> 3
- net SCK: track 6.47 -> 35.0 mm, vias 1 -> 4
- net CD: track 0.00 -> 28.3 mm, vias 0 -> 2
- net PORT_SERVO: track 0.00 -> 28.0 mm, vias 0 -> 1
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Other:
- board size 276.7 x 289.9 mm -> 57.6 x 40 mm

Commit message: fixed drc, the rest is bs
Routing:
- net +3.3V: track 267.5 -> 266.1 mm
Changed lines of the file:
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@@
+	)
+	(segment
+		(start 157.67 123.57)
+		(end 157.337652 123.902348)
+		(width 0.2)
+		(layer "F.Cu")
+		(net 1)
 	)
 	(segment
@@
 	)
 	(segment
-		(start 157.337652 123.49104)
-		(end 157.475515 123.353177)
-		(width 0.2)
-		(layer "F.Cu")
-		(net 1)
-	)
-	(segment
 		(start 191.412652 103.562652)
 		(end 192.537652 102.437652)
@@
 	)
 	(segment
+		(start 157.337652 123.902348)
+		(end 157.337652 124.437652)
+		(width 0.2)
+		(layer "F.Cu")
+		(net 1)
+	)
+	(segment
 		(start 149.200152 121.050152)
 		(end 149.087652 120.937652)
@@
 	)
 	(segment
-		(start 157.337652 124.437652)
-		(end 157.337652 123.49104)
-		(width 0.2)
-		(layer "F.Cu")
-		(net 1)
-	)
-	(segment
 		(start 173.937652 118.037652)
 		(end 173.937652 117.512652)
@@
 	)
 	(via
-		(at 157.475515 123.353177)
+		(at 157.67 123.57)
 		(size 0.6)
 		(drill 0.3)
@@
 		(width 0.2)
 		(layer "F.Cu")
-		(net 2)
-	)
-	(segment
-		(start 156.670152 121.537652)
-		(end 157.652652 122.520152)
-		(width 0.2)
-		(layer "F.Cu")
