File: vanguard/board versions/Vang_V2.3.4/Vanguard_new.kicad_pcb (KiCad board)
At the start: 4 copper layers, 40 x 50.3 mm, 99 parts, among them J1 USB_C_Receptacle_USB2.0_16P, J2 Micro_SD_Card_Det1, J3 Conn_02x03_Odd_Even, J4 Conn_01x03, J5 Conn_01x03, J6 Conn_01x03, J7 Conn_01x02_Pin, Q1 DMG2301L, Q4 BSS138, U1 TPS82130, U10 ATmega4809-A, U12 AP2112K-3.3, U3 ATSAMD11D14A-M, U4 BMP390L, U5 BD1020HFV-TR, U6 AT25DF641A-SH-T, U7 LTC4412xS6, U8 BNO055, U9 TPS61092, Y1 Crystal

Commit message: finished everything
Parts:
- moved TP6 1.08 mm to (139.4, 125.8)
- turned C26 to 90 degrees
Routing:
- net +3.3V: track 30.7 -> 261.8 mm, vias 10 -> 20
- net PORT_SERVO: track 0.00 -> 85.6 mm, vias 0 -> 2
- net STAR_SERVO: track 0.00 -> 78.1 mm
- net STAR_RED: track 0.00 -> 56.0 mm, vias 0 -> 5
- net PORT_RED: track 0.00 -> 53.8 mm, vias 0 -> 1
- net PORT_BLUE: track 0.00 -> 53.6 mm, vias 0 -> 1
- net +5V: track 9.98 -> 57.2 mm, vias 1 -> 3
- net PORT_GREEN: track 0.00 -> 45.7 mm, vias 0 -> 1
- net STAR_BLUE: track 0.00 -> 43.5 mm, vias 0 -> 3
- net EJEC_SERVO: track 0.00 -> 37.1 mm, vias 0 -> 2
- net TEMP_SENSOR: track 0.00 -> 33.7 mm, vias 0 -> 2
- net TX0: track 2.34 -> 33.8 mm, vias 1 -> 2
- net UPDI: track 14.1 -> 45.0 mm, vias 1 -> 2
- net RX0: track 1.98 -> 26.2 mm, vias 1 -> 3
- net STAR_GREEN: track 0.00 -> 22.7 mm, vias 0 -> 3
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Other:
- board size 40 x 50.3 mm -> 43.1 x 53.1 mm
