File: vanguard/board versions/Vang_V2.3.4/Vanguard_new.kicad_pcb (KiCad board)
At the start: 4 copper layers, 43.5 x 53.1 mm, 100 parts, among them J1 USB_C_Receptacle_USB2.0_16P, J2 Micro_SD_Card_Det1, J3 Conn_02x03_Odd_Even, J4 Conn_01x03, J5 Conn_01x03, J6 Conn_01x03, J7 Conn_01x02_Pin, Q1 DMG2301L, Q4 BSS138, U1 TPS82130, U10 ATmega4809-A, U12 AP2112K-3.3, U3 ATSAMD11D14A-M, U4 BMP390L, U5 BD1020HFV-TR, U6 AT25DF641A-SH-T, U7 LTC4412xS6, U8 BNO055, U9 TPS61092, Y1 32.768kHz

Commit message: edits
Changed lines of the file:
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@@
 		(tags "resistor")
 		(property "Reference" "R4"
-			(at 0 -1.43 135)
+			(at 3.667569 0.268701 135)
 			(layer "F.SilkS")
 			(effects
@@
 		(tags "capacitor")
 		(property "Reference" "C21"
-			(at 0.505 -1.84 270)
+			(at 0.205 -1.7 270)
 			(layer "F.SilkS")
 			(effects
@@
 		(tags "capacitor")
 		(property "Reference" "C11"
-			(at -2.1 0.68 180)
+			(at 2.48 -0.38 180)
 			(layer "F.SilkS")
 			(effects
@@
 		(tags "test point SMD pad rectangle square")
 		(property "Reference" "TP8"
-			(at 0 -1.448 0)
+			(at 3.75 -1.74 0)
 			(layer "F.SilkS")
 			(effects
@@
 		)
 		(fp_text user "${REFERENCE}"
-			(at 0 -1.45 0)
+			(at 3.76 -1.74 0)
 			(layer "F.Fab")
 			(effects
@@
 		(tags "resistor")
 		(property "Reference" "R22"
-			(at 1.695 3.345 0)
+			(at -0.185 -3.065 0)
 			(layer "F.SilkS")
 			(effects
@@
 		(tags "resistor")
 		(property "Reference" "R33"
-			(at 0 -1.429999 45)
+			(at 1.92333 1.513209 45)
 			(layer "F.SilkS")
 			(effects
@@
 		(tags "Buzzer Magnetic 9mm AT-0927-TT-6-R")
 		(property "Reference" "BZ1"
-			(at 2 5.5 0)
+			(at 1.97 1.96 0)
 			(layer "F.SilkS")
 			(effects
@@
 		(tags "['C26-LF']")
 		(property "Reference" "Y1"
-			(at 0.95 -2.23 0)
+			(at 0.85 2.34 0)
 			(layer "F.SilkS")
 			(effects
@@
 		(tags "resistor")
 		(property "Reference" "R23"
-			(at 3.765 2.875 0)
+			(at -3.485 -4.655 0)
 			(layer "F.SilkS")
 			(effects
@@
 		(tags "resistor")
 		(property "Reference" "R21"
-			(at 3.465 3.885 0)
+			(at 2.645 -1.565 0)
 			(layer "F.SilkS")
 			(effects
@@
 		(tags "SOT-143")
 		(property "Reference" "D2"
-			(at 0 0 315)
-			(layer "F.SilkS")
+			(at 0.307035 3.108793 -315)
+			(layer "B.SilkS")
 			(effects
 				(font
@@
 					(thickness 0.15)
 				)
+				(justify mirror)
 			)
 		)
@@
 		(tags "resistor")
 		(property "Reference" "R6"
-			(at 2.415 0.07 180)
+			(at 3.635 -0.09 180)
 			(layer "B.SilkS")
 			(effects

Commit message: production error
Parts:
- C26, C27: footprint Capacitor_SMD:C_0201_0603Metric -> Capacitor_SMD:C_0603_1608Metric
- D1, D13, D14, D3, D5: footprint LED_SMD:LED_0201_0603Metric -> LED_SMD:LED_0603_1608Metric
- moved D5 4.40 mm to (132.4, 91.1), turned to -135 degrees
- moved D3 2.26 mm to (136.9, 87.6)
- moved C6 1.93 mm to (144.9, 120.7), turned to 0 degrees
- moved D13 1.18 mm to (113.9, 86.3)
- moved D14 1.16 mm to (117.9, 96.7)
- moved C27 1.13 mm to (122.9, 106.4), turned to 90 degrees
- moved C26 0.76 mm to (120.4, 109.8)
- moved D1 0.44 mm to (138.2, 79.0)
Routing:
- net Net-(D5-A): track 1.24 -> 7.04 mm, vias 0 -> 2
- net RX0: track 26.2 -> 31.1 mm, vias 3 -> 4
- net TX0: track 35.8 -> 39.5 mm
- net GND: track 84.8 -> 88.0 mm, vias 50 -> 49
- net Net-(D3-A): track 1.29 -> 3.40 mm
- net +3.3V: track 263.0 -> 264.6 mm
- net Net-(D14-A): track 1.34 -> 2.05 mm
- net Net-(D13-A): track 1.30 -> 1.93 mm
