File: vanguard/board versions/Vang_V2.3.4/Vanguard_new.kicad_sch (KiCad schematic)
At the start: 99 parts, among them J1 USB_C_Receptacle_USB2.0_16P, J2 Micro_SD_Card_Det1, J3 Conn_02x03_Odd_Even, J4 Conn_01x03, J5 Conn_01x03, J6 Conn_01x03, J7 Conn_01x02_Pin, Q1 DMG2301L, Q4 BSS138, U1 TPS82130, U10 ATmega4809-A, U12 AP2112K-3.3, U3 ATSAMD11D14A-M, U4 BMP390L, U5 BD1020HFV-TR, U6 AT25DF641A-SH-T, U7 LTC4412xS6, U8 BNO055, U9 TPS61092, Y1 Crystal

Commit message: finished everything
Connections:
- net SWITCHOUT: now also D17.1 (K); no longer D17.2 (A)
- net VBUS: now also D17.2 (A); no longer D17.1 (K)
Other:
- moved on the sheet: D17, D3, D5, R11, R13
Changed lines of the file:
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@@
 	)
 	(junction
-		(at 228.6 77.47)
+		(at 208.28 74.93)
 		(diameter 0)
 		(color 0 0 0 0)
@@
 	)
 	(junction
-		(at 228.6 74.93)
+		(at 208.28 72.39)
 		(diameter 0)
 		(color 0 0 0 0)
@@
 	(wire
 		(pts
-			(xy 196.85 74.93) (xy 207.01 74.93)
+			(xy 196.85 74.93) (xy 208.28 74.93)
 		)
 		(stroke
@@
 	(wire
 		(pts
-			(xy 228.6 72.39) (xy 228.6 74.93)
+			(xy 208.28 69.85) (xy 208.28 72.39)
 		)
 		(stroke
@@
 	(wire
 		(pts
-			(xy 196.85 72.39) (xy 212.09 72.39)
+			(xy 196.85 72.39) (xy 208.28 72.39)
 		)
 		(stroke
@@
 	(wire
 		(pts
-			(xy 207.01 77.47) (xy 228.6 77.47)
-		)
-		(stroke
-			(width 0)
-			(type default)
-		)
-	)
-	(wire
-		(pts
 			(xy 146.05 40.64) (xy 166.37 40.64)
 		)
@@
 	(wire
 		(pts
-			(xy 207.01 74.93) (xy 207.01 77.47)
-		)
-		(stroke
-			(width 0)
-			(type default)
-		)
-	)
-	(wire
-		(pts
 			(xy 335.28 40.64) (xy 342.9 40.64)
 		)
@@
 	(wire
 		(pts
-			(xy 327.66 162.56) (xy 328.93 162.56)
+			(xy 326.39 162.56) (xy 328.93 162.56)
 		)
 		(stroke
@@
 	(wire
 		(pts
-			(xy 212.09 74.93) (xy 228.6 74.93)
-		)
-		(stroke
-			(width 0)
-			(type default)
-		)
-	)
-	(wire
-		(pts
 			(xy 156.21 233.68) (xy 157.48 233.68)
 		)
@@
 	(wire
 		(pts
-			(xy 228.6 77.47) (xy 234.95 77.47)
+			(xy 208.28 74.93) (xy 214.63 74.93)
 		)
 		(stroke
@@
 	(wire
 		(pts
-			(xy 228.6 77.47) (xy 228.6 80.01)
+			(xy 208.28 74.93) (xy 208.28 77.47)
 		)
 		(stroke
@@
 	(wire
 		(pts
-			(xy 212.09 72.39) (xy 212.09 74.93)
-		)
-		(stroke
-			(width 0)
-			(type default)
-		)
-	)
-	(wire
-		(pts
 			(xy 285.75 222.25) (xy 297.18 222.25)
 		)
@@
 	(wire
 		(pts
-			(xy 228.6 74.93) (xy 234.95 74.93)
+			(xy 208.28 72.39) (xy 214.63 72.39)
 		)
 		(stroke
@@
 	(global_label "TX0"
 		(shape output)
-		(at 234.95 77.47 0)
+		(at 214.63 74.93 0)
 		(fields_autoplaced yes)
 		(effects
@@
 		)
 		(property "Intersheetrefs" "${INTERSHEET_REFS}"
-			(at 241.3218 77.47 0)
+			(at 221.0018 74.93 0)
 			(effects
 				(font
@@
 	(global_label "RX0"
 		(shape input)
-		(at 234.95 74.93 0)
+		(at 214.63 72.39 0)
 		(fields_autoplaced yes)
 		(effects
@@
 		)
 		(property "Intersheetrefs" "${INTERSHEET_REFS}"
-			(at 241.6242 74.93 0)
+			(at 221.3042 72.39 0)
 			(effects
 				(font
@@
 	(global_label "SWITCHOUT"
 		(shape input)
-		(at 327.66 162.56 90)
+		(at 326.39 162.56 90)
 		(fields_autoplaced yes)
 		(effects
@@
 		)
 		(property "Intersheetrefs" "${INTERSHEET_REFS}"
-			(at 327.66 149.1124 90)
+			(at 326.39 149.1124 90)
 			(effects
 				(font
@@
 	(symbol
 		(lib_id "power:+3.3V")
-		(at 243.84 72.39 270)
+		(at 223.52 69.85 270)
 		(unit 1)
 		(exclude_from_sim no)
@@
 		(fields_autoplaced yes)
 		(property "Reference" "#PWR0148"
-			(at 240.03 72.39 0)
+			(at 219.71 69.85 0)
 			(effects
 				(font
@@
 		)
 		(property "Value" "+3.3V"
-			(at 248.92 72.39 0)
+			(at 228.6 69.85 0)
 			(effects
 				(font
@@
 		)
 		(property "Footprint" ""
-			(at 243.84 72.39 0)
+			(at 223.52 69.85 0)
 			(effects
 				(font
@@
 		)
 		(property "Datasheet" ""
-			(at 243.84 72.39 0)
+			(at 223.52 69.85 0)
 			(effects
 				(font
@@
 		)
 		(property "Description" "Power symbol creates a global label with name \"+3.3V\""
-			(at 243.84 72.39 0)
+			(at 223.52 69.85 0)
 			(effects
 				(font
@@
 	(symbol
 		(lib_id "Device:LED")
-		(at 232.41 72.39 0)
+		(at 212.09 69.85 0)
 		(unit 1)
 		(exclude_from_sim no)
@@
 		(dnp no)
 		(property "Reference" "D5"
-			(at 230.8225 80.01 0)
+			(at 210.5025 77.47 0)
 			(effects
 				(font
@@
 		)
 		(property "Value" "LED"
-			(at 231.648 68.072 0)
+			(at 211.328 65.532 0)
 			(effects
 				(font
@@
 		)
 		(property "Footprint" "LED_SMD:LED_0201_0603Metric"
-			(at 232.41 72.39 0)
+			(at 212.09 69.85 0)
 			(effects
 				(font
@@
 		)
 		(property "Datasheet" "~"
-			(at 232.41 72.39 0)
+			(at 212.09 69.85 0)
 			(effects
 				(font
@@
 		)
 		(property "Description" "Light emitting diode"
-			(at 232.41 72.39 0)
+			(at 212.09 69.85 0)
 			(effects
 				(font
@@
 		)
 		(property "Sim.Pins" "1=K 2=A"
-			(at 232.41 72.39 0)
+			(at 212.09 69.85 0)
 			(effects
 				(font
@@
 	(symbol
 		(lib_id "power:+3.3V")
-		(at 243.84 80.01 270)
+		(at 223.52 77.47 270)
 		(unit 1)
 		(exclude_from_sim no)
@@
 		(fields_autoplaced yes)
 		(property "Reference" "#PWR0163"
-			(at 240.03 80.01 0)
+			(at 219.71 77.47 0)
 			(effects
 				(font
@@
 		)
 		(property "Value" "+3.3V"
-			(at 248.92 80.01 0)
+			(at 228.6 77.47 0)
 			(effects
 				(font
@@
 		)
 		(property "Footprint" ""
-			(at 243.84 80.01 0)
+			(at 223.52 77.47 0)
 			(effects
 				(font
@@
 		)
 		(property "Datasheet" ""
-			(at 243.84 80.01 0)
+			(at 223.52 77.47 0)
 			(effects
 				(font
@@
 		)
 		(property "Description" "Power symbol creates a global label with name \"+3.3V\""
-			(at 243.84 80.01 0)
+			(at 223.52 77.47 0)
 			(effects
 				(font
@@
 	(symbol
 		(lib_id "Device:R")
-		(at 240.03 72.39 270)
+		(at 219.71 69.85 270)
 		(unit 1)
 		(exclude_from_sim no)
@@
 		(dnp no)
 		(property "Reference" "R13"
-			(at 240.03 72.39 90)
+			(at 219.71 69.85 90)
 			(effects
 				(font
@@
 		)
 		(property "Value" "330"
-			(at 240.284 70.104 90)
+			(at 219.964 67.564 90)
 			(effects
 				(font
@@
 		)
 		(property "Footprint" "Resistor_SMD:R_0603_1608Metric"
-			(at 240.03 70.612 90)
+			(at 219.71 68.072 90)
 			(effects
 				(font
@@
 		)
 		(property "Datasheet" "~"
-			(at 240.03 72.39 0)
+			(at 219.71 69.85 0)
 			(effects
 				(font
@@
 		)
 		(property "Description" "Resistor"
-			(at 240.03 72.39 0)
+			(at 219.71 69.85 0)
 			(effects
 				(font
@@
 	(symbol
 		(lib_id "Device:R")
-		(at 240.03 80.01 270)
+		(at 219.71 77.47 270)
 		(unit 1)
 		(exclude_from_sim no)
@@
 		(dnp no)
 		(property "Reference" "R11"
-			(at 240.03 80.01 90)
+			(at 219.71 77.47 90)
 			(effects
 				(font
@@
 		)
 		(property "Value" "330"
-			(at 240.284 82.296 90)
+			(at 219.964 79.756 90)
 			(effects
 				(font
@@
 		)
 		(property "Footprint" "Resistor_SMD:R_0603_1608Metric"
-			(at 240.03 78.232 90)
+			(at 219.71 75.692 90)
 			(effects
 				(font
@@
 		)
 		(property "Datasheet" "~"
-			(at 240.03 80.01 0)
+			(at 219.71 77.47 0)
 			(effects
 				(font
@@
 		)
 		(property "Description" "Resistor"
-			(at 240.03 80.01 0)
+			(at 219.71 77.47 0)
 			(effects
 				(font
@@
 	(symbol
 		(lib_id "Diode:PMEG6020ER")
-		(at 298.45 214.63 270)
+		(at 298.45 214.63 90)
 		(unit 1)
 		(exclude_from_sim no)
@@
 		(dnp no)
 		(property "Reference" "D17"
-			(at 288.29 216.916 0)
+			(at 308.61 212.344 0)
 			(effects
 				(font
@@
 		)
 		(property "Value" "PMEG6020ER"
-			(at 290.83 216.916 0)
+			(at 306.07 212.344 0)
 			(effects
 				(font
@@
 		)
 		(property "Footprint" "Diode_SMD:Nexperia_CFP3_SOD-123W"
-			(at 294.005 214.63 0)
+			(at 302.895 214.63 0)
 			(effects
 				(font
@@
 	(symbol
 		(lib_id "Device:LED")
-		(at 232.41 80.01 0)
+		(at 212.09 77.47 0)
 		(unit 1)
 		(exclude_from_sim no)
@@
 		(fields_autoplaced yes)
 		(property "Reference" "D3"
-			(at 230.8225 87.63 0)
+			(at 210.5025 85.09 0)
 			(effects
 				(font
@@
 		)
 		(property "Value" "LED"
-			(at 230.8225 85.09 0)
+			(at 210.5025 82.55 0)
 			(effects
 				(font
@@
 		)
 		(property "Footprint" "LED_SMD:LED_0201_0603Metric"
-			(at 232.41 80.01 0)
+			(at 212.09 77.47 0)
 			(effects
 				(font
@@
 		)
 		(property "Datasheet" "~"
-			(at 232.41 80.01 0)
+			(at 212.09 77.47 0)
 			(effects
 				(font
@@
 		)
 		(property "Description" "Light emitting diode"
-			(at 232.41 80.01 0)
+			(at 212.09 77.47 0)
 			(effects
 				(font
@@
 		)
 		(property "Sim.Pins" "1=K 2=A"
-			(at 232.41 80.01 0)
+			(at 212.09 77.47 0)
 			(effects
 				(font
