File: vanguard/meddy goof/Launch system/Vanguard_new.kicad_sch (KiCad schematic)
At the start: 74 parts, among them J1 USB_C_Receptacle_USB2.0_16P, J2 Micro_SD_Card_Det1, J3 Conn_02x03_Odd_Even, J5 igniter, Q4 BSS138, SW1 LAUNCH, SW2 POWER, SW4 SW_SPST, U1 TPS82130, U10 ATmega4809-A, U12 AP2112K-3.3, U2 SHT31-DIS, U3 ATSAMD11D14A-M, U4 BMP390L, U6 AT25DF641A-SH-T

Commit message: minor changes
Parts:
- removed BZ1: Buzzer, Buzzer_Beeper:MagneticBuzzer_Kingstate_KCG0601, symbol Device:Buzzer
- removed C26, C27: 0.1uF, Capacitor_SMD:C_0201_0603Metric, symbol Device:C
- removed C6, C7: 0.1uF, Capacitor_SMD:C_0603_1608Metric, symbol Device:C
- removed D1, D13, D3, D5: LED, LED_SMD:LED_0201_0603Metric, symbol Device:LED
- removed D12: PMEG6020ER, Diode_SMD:Nexperia_CFP3_SOD-123W, symbol Diode:PMEG6020ER
- removed D2: PRTR5V0U2X, Package_TO_SOT_SMD:SOT-143, symbol Power_Protection:PRTR5V0U2X
- removed D4, D6: LED, symbol Device:LED
- removed J1: USB_C_Receptacle_USB2.0_16P, Connector_USB:USB_C_Receptacle_Amphenol_124019772112A, symbol Connector:USB_C_Receptacle_USB2.0_16P
- removed J2: Micro_SD_Card_Det1, Connector_Card:microSD_HC_Hirose_DM3D-SF, symbol Connector:Micro_SD_Card_Det1
- removed J3: Conn_02x03_Odd_Even, Connector_PinHeader_2.54mm:PinHeader_2x03_P2.54mm_Vertical, symbol Connector_Generic:Conn_02x03_Odd_Even
- removed J5: igniter, symbol Connector:Conn_01x02_Pin
- removed JP1, JP2: Jumper_2_Small_Open, Jumper:SolderJumper-2_P1.3mm_Open_Pad1.0x1.5mm, symbol Jumper:Jumper_2_Small_Open
- removed JP3: SolderJumper_2_Open, symbol Jumper:SolderJumper_2_Open
- removed Q4: BSS138, Package_TO_SOT_SMD:SOT-23, symbol Transistor_FET:BSS138
- removed R13: 330, Resistor_SMD:R_0603_1608Metric, symbol Device:R
- removed R14: 4k7, Resistor_SMD:R_0603_1608Metric, symbol Device:R
- removed R15: R, symbol Device:R
- removed R16, R17: 10k, symbol Device:R
- removed R31: 10k, Resistor_SMD:R_0603_1608Metric, symbol Device:R
- removed R32, R33: 10k, Resistor_SMD:R_0201_0603Metric, symbol Device:R
- removed R34: 2k2, Resistor_SMD:R_0603_1608Metric, symbol Device:R
- removed SW1: LAUNCH, symbol Switch:SW_Push
- removed SW4: SW_SPST, symbol Switch:SW_SPST
- removed TP1, TP3, TP4, TP6: TestPoint, TestPoint:TestPoint_Pad_1.0x1.0mm, symbol Connector:TestPoint
- removed U1: TPS82130, Package_LGA:Texas_SIL0008D_MicroSiP-8-1EP_2.8x3mm_P0.65mm_EP1.1x1.9mm_ThermalVias, symbol Regulator_Switching:TPS82130
- removed U10: ATmega4809-A, Package_QFP:TQFP-48_7x7mm_P0.5mm, symbol MCU_Microchip_ATmega:ATmega4809-A
- removed U2: SHT31-DIS, Sensor_Humidity:Sensirion_DFN-8-1EP_2.5x2.5mm_P0.5mm_EP1.1x1.7mm, symbol Sensor_Humidity:SHT31-DIS
- removed U3: ATSAMD11D14A-M, Package_DFN_QFN:QFN-24-1EP_4x4mm_P0.5mm_EP2.6x2.6mm, symbol MCU_Microchip_SAMD:ATSAMD11D14A-M
- removed U6: AT25DF641A-SH-T, Package_SO:SOIC-8_3.9x4.9mm_P1.27mm, symbol AT25DF641A-SH-T:AT25DF641A-SH-T
- added A1: Arduino_Nano_Every, Module:Arduino_Nano, symbol MCU_Module:Arduino_Nano_Every
- added C22: C, Capacitor_SMD:C_0603_1608Metric, symbol Device:C
- added C6: 1000uF, symbol Device:C_Polarized_US
- added C7, C9: 100uF, symbol Device:C_Polarized_US
- added C8: 100n, symbol Device:C
- added D10, D8, D9: LED, symbol Device:LED
- added D11: 1N4007, symbol Device:D
- added D12, D13: D, symbol Device:D
- added D15: PMEG6020ER, Diode_SMD:Nexperia_CFP3_SOD-123W, symbol Diode:PMEG6020ER
- added D16, D17: LED, LED_SMD:LED_0201_0603Metric, symbol Device:LED
- added IC1: LM555N, symbol LM555N:LM555N
- added J3, J4: Conn_01x02_Pin, symbol Connector:Conn_01x02_Pin
- added L3: SLF7055T-6R8N2R8-3PF, Inductor_SMD:L_7.3x7.3_H4.5, symbol SLF7055T-6R8N2R8-3PF[1]:SLF7055T-6R8N2R8-3PF
- added SW10, SW7: SW_DPDT_x2, symbol Switch:SW_DPDT_x2
- added SW3: SW_DPST_x2, symbol Switch:SW_DPST_x2
- added SW8, SW9: SW_Push, symbol Switch:SW_Push
- added U1: TPS54308, Package_TO_SOT_SMD:SOT-23-6, symbol Regulator_Switching:TPS54308
- added U2: TPS82130, Package_LGA:Texas_SIL0008D_MicroSiP-8-1EP_2.8x3mm_P0.65mm_EP1.1x1.9mm_ThermalVias, symbol Regulator_Switching:TPS82130
- added U5: BD1020HFV-TR, Package_TO_SOT_SMD:HVSOF5, symbol Sensor_Temperature:BD1020HFV
- added U6: PC817, Package_DIP:DIP-4_W7.62mm, symbol Isolator:PC817
- C1: value 4n7 -> 0.1uF; footprint Capacitor_SMD:C_0603_1608Metric -> (none)
- C10: value 1uF -> 100n; footprint Capacitor_SMD:C_0603_1608Metric -> (none)
- C11: value 100nF -> 1uF
- C2: value 100n -> C; footprint Capacitor_SMD:C_0603_1608Metric -> (none)
- C3: value 0.1uF -> C
- C4: value 10uF -> C
- D14: footprint LED_SMD:LED_0201_0603Metric -> (none)
- R1, R2: value 10k -> R
- R10: value 4k7 -> 1k; footprint Resistor_SMD:R_0603_1608Metric -> (none)
- R11: value 330 -> 4k7
- R12: value 0 -> 4k7
- R3: value R -> 1k
- R35: value 350 -> 350k
- R4: value 330 -> R; footprint Resistor_SMD:R_0603_1608Metric -> (none)
- R5: value 5k1 -> R; footprint Resistor_SMD:R_0603_1608Metric -> (none)
- R6: value 5k1 -> 2k2; footprint Resistor_SMD:R_0603_1608Metric -> (none)
- R7: value 4k7 -> 2k2; footprint Resistor_SMD:R_0603_1608Metric -> (none)
- R8: value 4k7 -> 470; footprint Resistor_SMD:R_0603_1608Metric -> (none)
- R9: value 4k7 -> R; footprint Resistor_SMD:R_0603_1608Metric -> (none)
- SW2: value POWER -> SW_SPDT
Connections:
- net RX_UPDI is gone; now on net +3.3V: R12.1
- net UPDI is gone; now on net SCL: R12.2
- net +3.3V: now also U4.5 (SDO/DNC/SA0), C22.2, U5.4 (VDD); no longer C11.2, C3.1, C4.1, R1.1, R10.2, R7.1, R8.1, R9.1
- net GND: now also C11.2, C2.2, C4.2, R3.2, R4.2, A1.20 (A1), A1.29 (GND), A1.4 (GND), C22.1, C6.2, C7.2, C8.2, C9.2, D16.1 (K), D17.1 (K), D8.1 (K), D9.1 (K), IC1.1 (GND), J3.2 (Pin_2), J4.1 (Pin_1), U1.5 (EN), U2.3 (GND), U2.9 (GND), U5.2 (PG), U5.5 (GND), U6.3; no longer C11.1, C2.1, R5.2, R6.2
- net SCL: now also A1.24 (SCL/A5)
- net SDA: now also R11.2, A1.23 (SDA/A4); no longer R10.1, R7.2
- net at D14.2 (A): now also R10.1; no longer R39.2
- net at R8.2: now also D10.2 (A)
- net at C14.1: now also D15.1 (K), U2.1 (EN), U2.2 (VIN)
- net at C16.1, R35.1, R38.1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: now also C11.1, U2.4 (VOUT), U2.5 (VOUT); no longer C10.1
- net at R38.2: now also D16.2 (A)
- net +5V: now reaches R4.1
- net +5V: now also C1.2, C4.1, R1.1, R5.1, A1.30 (VIN), D15.2 (A), L3.2
- net at R2.1: now also R1.2, U1.4 (FB)
- net at R3.1: now also U6.1
- net at R9.2: now also C7.1, IC1.2 (TR), IC1.6 (THR)
- net at R35.2, R37.1: now also U2.6 (FB)
- net at BZ2.1 (+): now also R10.2, D13.1 (K)
- net at C15.1: now also U2.8 (SS/TR)
- net at SW2.1 (A): now also R6.1, C6.1, SW7.2 (B), SW8.1
- net at C3.2: now also L3.1, U1.2 (SW)
- removed net VBUS: C1.2, C2.2, R4.2, SW2.2 (B)
- net pwr: no longer names the net of SW2.3 (C)
- new net: C10.1, IC1.5 (CV)
- new net: D9.2 (A), R7.2
- new net: C8.1, C9.1, D11.1 (K), D12.1 (K), IC1.4 (~{RST}), IC1.8 (V+), R9.1
- new net: D12.2 (A), D13.2 (A), IC1.3 (Q)
- new net: R8.1, SW8.2
- new net: D11.2 (A), SW9.2
- new net: C3.1, U1.6 (BOOT)
- new net: J3.1 (Pin_1), SW3.1 (A)
- new net: D10.1 (K), J4.2 (Pin_2), SW10.1 (A), U6.2
- new net: R5.2, U6.4
- new net: D8.2 (A), R6.2
- new net: D17.2 (A), R39.2
- new net: R7.1, SW10.2 (B), SW7.3 (C), SW9.1
- new net BAT+: C2.1, SW2.2 (B), SW3.2 (B), U1.3 (VIN)
- new net temp_sens: A1.19 (A0), U5.3 (OUT)
- no-connect marks 26 -> 0
Other:
- note removed: "BUZZER"
- note removed: "FLASH CHIP"
- note removed: "INPUT USB"
- note removed: "LEDS"
- note removed: "POWER STABILIZATION"
- note removed: "SD CARD"
- moved on the sheet: C14, C15, C16, C18, C20, C21, R35, R37, R38, R39, U12, U4

Commit message: e
Parts:
- removed SW8: SW_Push, symbol Switch:SW_Push
- added SW4: SW_DPST_x2, Connector_PinHeader_2.54mm:PinHeader_1x02_P2.54mm_Vertical, symbol Switch:SW_DPST_x2
- BZ2: footprint (none) -> Buzzer_Beeper:Buzzer_12x9.5RM7.6
- C1, C10, C6, C7, C8, C9: footprint (none) -> Capacitor_SMD:C_0805_2012Metric
- C11, C14, C15, C16, C18, C20, C21: footprint Capacitor_SMD:C_0603_1608Metric -> Capacitor_SMD:C_0805_2012Metric
- C2: value C -> 10uF; footprint (none) -> Capacitor_SMD:C_0805_2012Metric
- C22: value C -> 0.1uF; footprint Capacitor_SMD:C_0603_1608Metric -> Capacitor_SMD:C_0805_2012Metric
- C3: value C -> 0.1uF; footprint (none) -> Capacitor_SMD:C_0805_2012Metric
- C4: value C -> 1nF; footprint (none) -> Capacitor_SMD:C_0805_2012Metric
- D10, D14, D8, D9: footprint (none) -> LED_THT:LED_D3.0mm
- D11: footprint (none) -> Diode_SMD:D_SOD-123F
- D12, D13: value D -> 1N4007; footprint (none) -> Diode_SMD:D_SOD-123F
- IC1: footprint (none) -> Package_SO:SOIC-8_3.9x4.9mm_P1.27mm
- J3: footprint (none) -> Connector_AMASS:AMASS_XT60-F_1x02_P7.20mm_Vertical
- J4: footprint (none) -> Connector_PinSocket_2.54mm:PinSocket_1x02_P2.54mm_Vertical
- R1: value R -> 52.3k; footprint (none) -> Resistor_SMD:R_0805_2012Metric
- R10, R3, R4, R5, R6, R7, R8: footprint (none) -> Resistor_SMD:R_0805_2012Metric
- R11, R12, R35, R37, R38, R39: footprint Resistor_SMD:R_0603_1608Metric -> Resistor_SMD:R_0805_2012Metric
- R2, R9: value R -> 10k; footprint (none) -> Resistor_SMD:R_0805_2012Metric
- SW10, SW2, SW7: footprint (none) -> Connector_PinHeader_2.54mm:PinHeader_1x03_P2.54mm_Vertical
- SW3, SW9: footprint (none) -> Connector_PinHeader_2.54mm:PinHeader_1x02_P2.54mm_Vertical
Connections:
- net at C6.1, R6.1, SW2.1 (A)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: now also SW4.1 (A)
- net at R8.1: now also SW4.2 (B)
Other:
- moved on the sheet: BZ2, C10, C6, C7, C8, C9, D10, D11, D12, D13, D14, D8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
