File: vanguard/board versions/Vang_V2.3.5/Vanguard_new.kicad_sch (KiCad schematic)
At the start: 99 parts, among them J1 USB_C_Receptacle_USB2.0_16P, J2 Micro_SD_Card_Det1, J3 Conn_02x03_Odd_Even, J4 Conn_01x03, J5 Conn_01x03, J6 Conn_01x03, J7 Conn_01x02_Pin, Q1 DMG2301L, Q4 BSS138, U1 TPS82130, U10 ATmega4809-A, U12 AP2112K-3.3, U3 ATSAMD11D14A-M, U4 BMP390L, U5 BD1020HFV-TR, U6 AT25DF641A-SH-T, U7 LTC4412xS6, U8 BNO055, U9 TPS61092, Y1 32.768kHz

Commit message: bom + minor fixes
Parts:
- added C24, C9: 22pF, symbol Device:C_Polarized_US
- added C28, C29: 100nF, Capacitor_SMD:C_0603_1608Metric, symbol Device:C
- added C30, C31, C32: 0.1uF, symbol Device:C_Polarized_US
- added R14, R15, R16, R17: 2k2, Resistor_SMD:R_0603_1608Metric, symbol Device:R
- added R18, R19: R, symbol Device:R
- added TP10, TP11: TestPoint, TestPoint:TestPoint_Pad_1.0x1.0mm, symbol Connector:TestPoint
- added U11: lsm6dso32, Package_LGA:LGA-14_3x2.5mm_P0.5mm_LayoutBorder3x4y, symbol Sensor_Motion:LSM6DS3
- added U2: BNO086, BNO086:IC_BNO086, symbol BNO086:BNO086
- added Y2: Crystal, symbol Device:Crystal
- BZ1: footprint Buzzer_Beeper:MagneticBuzzer_PUI_AT-0927-TT-6-R -> Buzzer_Beeper:MagneticBuzzer_Kingstate_KCG0601
- C13: footprint Capacitor_THT:CP_Radial_D4.0mm_P2.00mm -> Capacitor_SMD:C_0603_1608Metric
- C17, C19, C20, C21, C3, C6, C7: value 100nF -> 0.1uF
- C22: value 100nF -> C
- C26, C27: value 100nF -> 0.1uF; footprint Capacitor_SMD:C_0201_0603Metric -> Capacitor_SMD:C_0603_1608Metric
- R32, R33: footprint Resistor_SMD:R_0603_1608Metric -> Resistor_SMD:R_0201_0603Metric
- Y1: value 32.768kHz -> Crystal
Connections:
- net +3.3V: now also C22.2, C28.1, C29.1, C31.1, C32.1, R14.1, R15.1, R16.1, R17.1, R18.1, U11.5 (VDDIO), U11.8 (VDD), U2.18 (~{H_CS}), U2.28 (VDDIO), U2.3 (VDD), U2.6 (PS0/WAKE); no longer C22.1
- net GND: now also C22.1, C24.2, C28.2, C29.2, C30.2, C31.2, C32.2, C9.2, R19.2, U11.6 (GND), U11.7 (GND), U2.2 (GND), U2.25 (GNDIO), U2.5 (PS1); no longer C22.2
- net SCL: now also R14.2, TP10.1, U11.13 (SCL), U2.19 (H_SCL/SCK/RX)
- net SDA: now also R15.2, R16.2, R17.2, TP11.1, U11.14 (SDA), U2.20 (H_SDA/H_MISO/TX)
- new net: C24.1, U2.27 (XIN32), Y2.1
- new net: U2.1 (RESV_NC), U2.12 (RESV_NC), U2.13 (RESV_NC), U2.21 (RESV_NC), U2.22 (RESV_NC), U2.23 (RESV_NC), U2.24 (RESV_NC), U2.7 (RESV_NC), U2.8 (RESV_NC)
- new net: R18.2, R19.1, U2.17 (SA0/H_MOSI)
- new net: C9.1, U2.26 (XOUT32/CLKSEL1), Y2.2
- new net: C30.1, U2.9 (CAP)
Other:
- moved on the sheet: R12

Commit message: edits
Parts:
- removed C24, C9: 22pF, symbol Device:C_Polarized_US
- removed C28, C29: 100nF, Capacitor_SMD:C_0603_1608Metric, symbol Device:C
- removed C30, C31, C32: 0.1uF, symbol Device:C_Polarized_US
- removed R14, R15, R16, R17: 2k2, Resistor_SMD:R_0603_1608Metric, symbol Device:R
- removed R18, R19: R, symbol Device:R
- removed TP10, TP11: TestPoint, TestPoint:TestPoint_Pad_1.0x1.0mm, symbol Connector:TestPoint
- removed U11: lsm6dso32, Package_LGA:LGA-14_3x2.5mm_P0.5mm_LayoutBorder3x4y, symbol Sensor_Motion:LSM6DS3
- removed U2: BNO086, BNO086:IC_BNO086, symbol BNO086:BNO086
- removed Y2: Crystal, symbol Device:Crystal
- BZ1: footprint Buzzer_Beeper:MagneticBuzzer_Kingstate_KCG0601 -> Buzzer_Beeper:MagneticBuzzer_PUI_AT-0927-TT-6-R
- C13: footprint Capacitor_SMD:C_0603_1608Metric -> Capacitor_THT:CP_Radial_D4.0mm_P2.00mm
- C17, C19, C20, C21, C3, C6, C7: value 0.1uF -> 100nF
- C22: value C -> 100nF
- C26, C27: value 0.1uF -> 100nF; footprint Capacitor_SMD:C_0603_1608Metric -> Capacitor_SMD:C_0201_0603Metric
- R32, R33: footprint Resistor_SMD:R_0201_0603Metric -> Resistor_SMD:R_0603_1608Metric
- Y1: value Crystal -> 32.768kHz
Connections:
- net +3.3V: now also C22.1; no longer C22.2
- net GND: now also C22.2; no longer C22.1
Other:
- moved on the sheet: R12
